File: ESP32S3_Audio_Cam_POE.kicad_sch (KiCad schematic)
At the start: 219 parts, among them J1 USB-C, J10 Conn_01x02, J11 Conn_01x02, J2 HC-RJ45-055-4_8P8C_Shielded, J3 Conn_01x02, J4 Conn_01x03, J5 Conn_01x03, J6 Conn_01x03, J7 Conn_01x02, J8 Conn_01x03, J9 Conn_01x02, Q1 AO3401A, Q2 AO3401A, Q3 AO3401A, Q4 AO3401A, Q5 AO3401A, T1 H1102NLT, U1 USBLC6-2SC6, U10 MAX98357AETE+T, U11 ICS-43434, U12 DS18B20U(UMW), U13 ESP32-S3, U2 TLV62568DBVR, U3 IR26-21C/L110/CT, U4 W25Q128, U5 W5500, U6 DP9900M-5V, U7 XC6206-2.8V, U8 XC6206-1.5NR, U9 TM1637, X1 X322525MOB4SI, Y1 40MHz, Y2 32.768KHz

Commit message: draft commit
Parts:
- added C59, C60: 100nF, PCM_JLCPCB:C_0603, symbol PCM_JLCPCB-Capacitors:0603,100nF
- added U14: TCA9535PWR, JLCPCB:port-expander-I2C_TCA9535PWR_C130204, symbol JLCPCB-Extended:TCA9535PWR_C130204
- added U15: MT9221CT-06BR5, JLCPCB:Current-sensor_MT9221CT-06BR5_C879632, symbol JLCPCB-Extended:Current-sensor_MT9221CT-06BR5_C879632
Connections:
- net +3V3: now also C59.1, U14.24 (VCC)
- net Earth: now also C59.2, C60.2, U14.12 (GND), U15.5 (GND)
- net VBUS: now also C60.1, U15.1 (IP+), U15.2 (IP+), U15.8 (VCC); no longer C6.1, R5.1, TP3.1, U2.4 (VIN)
- new net ISEN.FLT: U15.6 (FILTER)
- new net ISEN.VO: U15.7 (VOUT)
- new net PORT.SCL: U14.22 (SCL)
- new net PORT.SDA: U14.23 (SDA)
- new net Vdrive: C6.1, R5.1, TP3.1, U15.3 (IP-), U15.4 (IP-), U2.4 (VIN)

Commit message: draft check in
Parts:
- removed U14: TCA9535PWR, JLCPCB:port-expander-I2C_TCA9535PWR_C130204, symbol JLCPCB-Extended:TCA9535PWR_C130204
- added BOOT2: SW_BOOT, Button_Switch_SMD:SW_SPST_EVQP2, symbol Switch:SW_Push
- added C61: 1uF, PCM_JLCPCB:C_0603, symbol PCM_JLCPCB-Capacitors:0603,1uF
- added C62, C63, C64, C65, C66: 100nF, PCM_JLCPCB:C_0603, symbol PCM_JLCPCB-Capacitors:0603,100nF
- added C67, C68: 10pF, PCM_JLCPCB:C_0402, symbol PCM_JLCPCB-Capacitors:0402,10pF
- added C69, C70: 20pF, PCM_JLCPCB:C_0402, symbol PCM_JLCPCB-Capacitors:0402,20pF
- added J12: Conn_01x02, Connector_PinHeader_1.00mm:PinHeader_1x02_P1.00mm_Vertical, symbol Connector_Generic:Conn_01x02
- added JP5: SolderJumper_3_Bridged12, symbol Jumper:SolderJumper_3_Bridged12
- added JP6, JP7: Jumper_2_Small_Bridged, Jumper:SolderJumper-2_P1.3mm_Bridged_RoundedPad1.0x1.5mm, symbol Jumper:Jumper_2_Small_Bridged
- added R59: 10kΩ, PCM_JLCPCB:R_0402, symbol PCM_JLCPCB-Resistors:0402,10kΩ
- added R60: 22Ω, PCM_JLCPCB:R_0402, symbol PCM_JLCPCB-Resistors:0402,22Ω
- added RST2: SW_RST, Button_Switch_SMD:SW_SPST_EVQP2, symbol Switch:SW_Push
- added TP1: TestPoint, TestPoint:TestPoint_Pad_D1.0mm, symbol Connector:TestPoint
- added U16: ESP32-S3, PCM_JLCPCB:QFN-56-1EP_7x7mm_P0.4mm_EP4x4mm_ThermalVias, symbol PCM_JLCPCB-Extended:MCU, ESP32-S3
- added Y3: 40MHz, Crystal:Crystal_SMD_3225-4Pin_3.2x2.5mm, symbol Device:Crystal_GND24
- added Y4: 32.768KHz, Crystal:Crystal_SMD_3215-2Pin_3.2x1.5mm, symbol Device:Crystal
Connections:
- net MIC.SCK is gone; now on net GPIO35: U11.4 (SCK)
- net MIC.SD is gone; now on net GPIO34: U11.6 (SD)
- net MIC.WS is gone; now on net GPIO33: U11.1 (WS), U12.1 (DQ)
- net SPK.BCLK is gone; now on net GPIO37: U10.16 (BCLK)
- net SPK.DIN is gone; now on net GPIO36: U10.1 (DIN)
- net SPK.LRCLK is gone; now on net GPIO21: U10.14 (LRCLK)
- net +3V3: now also C61.1, C62.2, C63.2, C64.2, C65.2, JP5.3 (B), R59.2, TP1.1, U16.2 (VDD3P3), U16.20 (VDD3P3_RTC), U16.3 (VDD3P3), U16.55 (VDDA), U16.56 (VDDA); no longer C59.1
- net +3V3_RF: now also U16.46 (VDD3P3_CPU)
- net Earth: now also C59.1, BOOT2.1, C61.2, C62.1, C63.1, C64.1, C65.1, C66.1, C67.2, C68.2, C69.2, C70.2, JP5.1 (A), RST2.1, U16.57 (GND), Y3.2, Y3.4; no longer C59.2
- net GPIO21: no longer D10.4 (DIN), TP10.1
- net GPIO43: now also JP7.1 (A)
- net GPIO44: now also JP6.1 (A)
- net MIC.LR: now also JP5.2 (C)
- net VDD_SPI: now also U16.29 (VDD_SPI)
- net 7SEG.CLK renamed 2GPIO2
- net 2GPIO2: now also U16.7 (GPIO2)
- net 7SEG.DIO renamed 2GPIO3
- net 2GPIO3: now also U16.8 (GPIO3)
- net ISEN.VO renamed 2GPIO17
- net 2GPIO17: now also U16.23 (GPIO17)
- net LED.IR renamed 2GPIO5
- net 2GPIO5: now also U16.10 (GPIO5)
- net LED.OTH renamed 2GPIO6
- net 2GPIO6: now also U16.11 (GPIO6)
- net LED.WH renamed 2GPIO4
- net 2GPIO4: now also U16.9 (GPIO4)
- net RC.OTHR renamed 2GPIO12
- net 2GPIO12: now also U16.17 (GPIO12)
- net RC.PAN renamed 2GPIO9
- net 2GPIO9: now also U16.14 (GPIO9)
- net RC.ROT renamed 2GPIO11
- net 2GPIO11: now also U16.16 (GPIO11)
- net RC.TILT renamed 2GPIO10
- net 2GPIO10: now also U16.15 (GPIO10)
- new net: C67.1, R60.1, Y3.1
- new net 2CHIP_BOOT: BOOT2.2, C66.2, U16.5 (GPIO0)
- new net 2CHIP_PU: C59.2, R59.1, RST2.2, U16.4 (CHIP_PU)
- new net 2GPIO1: U16.6 (GPIO1)
- new net 2GPIO13: U16.18 (GPIO13)
- new net 2GPIO14: U16.19 (GPIO14)
- new net 2GPIO15: C69.1, U16.21 (XTAL_32K_P), Y4.1
- new net 2GPIO16: C70.1, U16.22 (XTAL_32K_N), Y4.2
- new net 2GPIO18: U16.24 (GPIO18)
- new net 2GPIO19: U16.25 (GPIO19/USB_D-)
- new net 2GPIO20: U16.26 (GPIO20/USB_D+)
- new net 2GPIO21: U16.27 (GPIO21)
- new net 2GPIO26: U16.28 (SPICS1)
- new net 2GPIO27: U16.30 (SPIHD)
- new net 2GPIO28: U16.31 (SPIWP)
- new net 2GPIO29: U16.32 (SPICS0)
- new net 2GPIO30: U16.33 (SPICLK)
- new net 2GPIO31: U16.34 (SPIQ)
- new net 2GPIO32: U16.35 (SPID)
- new net 2GPIO33: U16.38 (GPIO33)
- new net 2GPIO34: U16.39 (GPIO34)
- new net 2GPIO35: U16.40 (GPIO35)
- new net 2GPIO36: U16.41 (GPIO36)
- new net 2GPIO37: U16.42 (GPIO37)
- new net 2GPIO38: U16.43 (GPIO38)
- new net 2GPIO39: U16.44 (MTCK)
- new net 2GPIO40: U16.45 (MTDO)
- new net 2GPIO41: U16.47 (MTDI)
- new net 2GPIO42: U16.48 (MTMS)
- new net 2GPIO43: J12.1 (Pin_1), JP6.2 (B), U16.49 (U0TXD)
- new net 2GPIO44: J12.2 (Pin_2), JP7.2 (B), U16.50 (U0RXD)
- new net 2GPIO45: U16.51 (GPIO45)
- new net 2GPIO46: U16.52 (GPIO46)
- new net 2GPIO47: U16.37 (SPICLK_P)
- new net 2GPIO48: U16.36 (SPICLK_N)
- new net 2GPIO7: U16.12 (GPIO7)
- new net 2GPIO8: U16.13 (GPIO8)
- new net 2OSC_IN: R60.2, U16.54 (XTAL_P)
- new net 2OSC_OUT: C68.1, U16.53 (XTAL_N), Y3.3
- new net LED.RGB: D10.4 (DIN), TP10.1
Other:
- moved on the sheet: ANT1, BOOT1, C10, C11, C12, C13, C14, C15, C16, C17, C18, C19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

Commit message: Draft commit, needs routing, schematic is probably mostly OK. Footprints are roughly located.
Parts:
- removed C11: 1uF, PCM_JLCPCB:C_0603, symbol PCM_JLCPCB-Capacitors:0603,1uF
- removed C13, C14, C16, C18, C59, C66: 100nF, PCM_JLCPCB:C_0603, symbol PCM_JLCPCB-Capacitors:0603,100nF
- removed C22, C24: 20pF, PCM_JLCPCB:C_0402, symbol PCM_JLCPCB-Capacitors:0402,20pF
- removed R59: 10kΩ, PCM_JLCPCB:R_0402, symbol PCM_JLCPCB-Resistors:0402,10kΩ
- removed TP1, TP43: TestPoint, TestPoint:TestPoint_Pad_D1.0mm, symbol Connector:TestPoint
- removed Y2: 32.768KHz, Crystal:Crystal_SMD_3215-2Pin_3.2x1.5mm, symbol Device:Crystal
- added C2: 1nF, PCM_JLCPCB:C_0402, symbol JLCPCB-Capacitors:0402,1nF
- added C23, C42: 1uF, PCM_JLCPCB:C_0603, symbol PCM_JLCPCB-Capacitors:0603,1uF
- added C24, C25, C27, C30, C41, C57, C69, C72: 100nF, PCM_JLCPCB:C_0603, symbol PCM_JLCPCB-Capacitors:0603,100nF
- added D2: 1N4148W, PCM_JLCPCB:D_SOD-123, symbol PCM_JLCPCB-Diodes:Switching,1N4148W
- added J2: USB-C, Connector_USB:USB_C_Receptacle_GCT_USB4105-xx-A_16P_TopMnt_Horizontal, symbol PCB_Lib_DaanHeetkamp:USB_C_Receptacle_USB2.0
- added JP8: SolderJumper_3_Bridged12, Jumper:SolderJumper-3_P1.3mm_Bridged12_Pad1.0x1.5mm, symbol Jumper:SolderJumper_3_Bridged12
- added PB2, RST2: SW_RST, Button_Switch_SMD:SW_SPST_EVQP2, symbol Switch:SW_Push
- added R12, R13: 33Ω, PCM_JLCPCB:R_0402, symbol PCM_JLCPCB-Resistors:0402,33Ω
- added R33: 100kΩ, PCM_JLCPCB:R_0402, symbol PCM_JLCPCB-Resistors:0402,100kΩ
- added R5, R7: 5.1kΩ, PCM_JLCPCB:R_0402, symbol PCM_JLCPCB-Resistors:0402,5.1kΩ
- added R52: 10kΩ, PCM_JLCPCB:R_0402, symbol PCM_JLCPCB-Resistors:0402,10kΩ
- added TP16, TP17, TP18, TP19, TP20, TP21, TP22, TP23, TP24, TP25, TP26, TP27, TP28, TP29, TP30, TP31, TP32, TP4, TP49, TP5, TP6, TP8, TP9: TestPoint, TestPoint:TestPoint_Pad_D1.0mm, symbol Connector:TestPoint
- added TST-R1, TST-R10, TST-R11, TST-R12, TST-R13, TST-R14, TST-R15, TST-R16, TST-R17, TST-R18, TST-R19, TST-R2, TST-R20, TST-R21, TST-R22, TST-R23, TST-R24, TST-R25, TST-R26, TST-R27, TST-R3, TST-R4, TST-R5, TST-R6, TST-R7, TST-R8, TST-R9: 0Ω, PCM_JLCPCB:R_0603, symbol PCM_JLCPCB-Resistors:0603,0Ω
- added U10: W25Q128, PCM_JLCPCB:SOIC-8_L5.3-W5.3-P1.27-LS8.0-BL, symbol PCM_JLCPCB-Memory:16MByte, SPI
- added U17: ICS-43434, JLCPCB:ICS-43434_C5656610, symbol JLCPCB-ICs:ICS-43434_C5656610
- added U4: USBLC6-2SC6, Package_TO_SOT_SMD:SOT-23-6, symbol Power_Protection:USBLC6-2SC6
- D13: renamed from U3; value IR26-21C/L110/CT -> IR
- JP7: renamed from JP5; footprint (none) -> Jumper:SolderJumper-3_P1.3mm_Bridged12_Pad1.0x1.5mm
- TP45: renamed from TP36; footprint TestPoint:TestPoint_Plated_Hole_D2.0mm -> TestPoint:TestPoint_Pad_D1.0mm
- TP46: renamed from TP37; footprint TestPoint:TestPoint_Plated_Hole_D2.0mm -> TestPoint:TestPoint_Pad_D1.0mm
- TP47: renamed from TP38; footprint TestPoint:TestPoint_Plated_Hole_D2.0mm -> TestPoint:TestPoint_Pad_D1.0mm
- U5: renamed from U8; footprint PCM_JLCPCB:SOT-23-3_L2.9-W1.6-P1.90-LS2.8-BR -> Package_TO_SOT_SMD:SOT-23-3; symbol XC6206-1.5V:LDO, 1.5V, 0.2A -> JLCPCB-ICs:XC6206-1.5NR C2984869
- U6: renamed from U7; footprint PCM_JLCPCB:SOT-23-3_L2.9-W1.6-P1.90-LS2.8-BR -> Package_TO_SOT_SMD:SOT-23-3; symbol XC6206-2.8V:LDO, 2.8V, 0.2A -> JLCPCB-ICs:XC6206-2.8V_C2892669
- renumbered C6 to C1, C70 to C10, C8 to C11, C9 to C13, C10 to C14, C46 to C16, C47 to C17, C48 to C18, C44 to C19, C43 to C20, C41 to C21, C42 to C22, C61 to C26, C62 to C28, C63 to C29, C19 to C3, C64 to C31, C65 to C32, C1 to C33, C2 to C34, C28 to C35, C27 to C36, C5 to C37, C45 to C38, C4 to C39, C67 to C4, C3 to C40, C49 to C43, C50 to C44, C51 to C45, C17 to C46, C52 to C47, C20 to C48, C58 to C49, C60 to C5, C29 to C50, C30 to C51, C32 to C52, C31 to C53, C56 to C54, C25 to C56, C23 to C58, C35 to C59, C21 to C6, C33 to C60, C39 to C61, C36 to C62, C34 to C63, C40 to C64, C38 to C65, C54 to C66, C53 to C67, C26 to C68, C68 to C7, C37 to C70, C57 to C71, C7 to C8, C69 to C9, D9 to D1, D2 to D10, D8 to D11, D11 to D12, D6 to D5, D7 to D6, D5 to D7, D1 to D8, D10 to D9, LED2 to DISP1, J7 to J10, J9 to J11, J10 to J12, J11 to J13, J12 to J4, J4 to J5, J5 to J6, J6 to J7, J2 to J9, JP6 to JP1, JP7 to JP2, JP1 to JP5, JP2 to JP6, RST2 to PB1, R9 to R1, R4 to R10, R3 to R11, R34 to R14, R35 to R15, R37 to R16, R38 to R17, R39 to R18, R36 to R19, R60 to R2, R13 to R20, R14 to R21, R19 to R22, R20 to R23, R21 to R24, R22 to R25, R23 to R26, R24 to R27, R16 to R28, R40 to R29, R5 to R3, R41 to R30, R42 to R31, R43 to R32, R17 to R34, R18 to R35, R15 to R36, R8 to R37, R47 to R38, R46 to R39, R1 to R4, R50 to R40, R49 to R41, R44 to R42, R48 to R43, R27 to R44, R28 to R45, R29 to R46, R45 to R47, R25 to R48, R26 to R49, R11 to R50, R10 to R51, R12 to R53, R51 to R54, R53 to R55, R55 to R56, R52 to R57, R54 to R58, R33 to R59, R2 to R6, R32 to R60, R31 to R61, R30 to R62, R56 to R63, R58 to R64, R57 to R65, R6 to R8, R7 to R9, TP3 to TP1, TP27 to TP11, TP28 to TP12, TP29 to TP13, TP30 to TP14, TP31 to TP15, TP4 to TP2, TP5 to TP3, TP16 to TP33, TP17 to TP34, TP18 to TP35, TP19 to TP36, TP20 to TP37, TP21 to TP38, TP22 to TP39, TP23 to TP40, TP24 to TP41, TP25 to TP42, TP26 to TP43, TP41 to TP48, TP42 to TP50, TP32 to TP51, TP34 to TP52, TP33 to TP53, TP35 to TP54, TP12 to TP55, TP13 to TP56, TP40 to TP57, TP39 to TP58, TP8 to TP59, TP9 to TP60, TP14 to TP61, TP15 to TP62, TP10 to TP63, TP45 to TP64, TP46 to TP65, TP11 to TP66, TP47 to TP67, TP48 to TP68, U2 to U1, U9 to U11, U4 to U13, U6 to U14, U10 to U15, U11 to U16, U15 to U2, U1 to U3, U13 to U7, U16 to U8, U5 to U9, Y3 to Y2, Y4 to Y3
Connections:
- net 2GPIO13 is gone; now on net RC.OTHR: U8.18 (GPIO13)
- net 2GPIO21 is gone; now on net LED.RGB: U8.27 (GPIO21)
- net 2GPIO29 is gone; now on net 2FLASH_QSPI_nCS: U8.32 (SPICS0)
- net GPIO17 is gone; now on net CAM.D6: U7.23 (GPIO17)
- net +1V5: now also TST-R8.2; no longer C17.1, C19.2, U5.2 (VOUT)
- net +2V8: now also TST-R9.2; no longer C18.1, C20.2, U6.2 (VOUT)
- net +3V3: now also R52.2, TST-R10.2, TST-R11.2, TST-R12.2, TST-R13.2, TST-R14.2, TST-R15.1, TST-R19.2, TST-R2.2, TST-R20.2, TST-R25.2, TST-R26.2, TST-R27.2, TST-R6.2, TST-R7.1; no longer C26.1, C28.2, C29.2, C31.2, C32.2, C35.2, C38.2, C43.2, C44.1, C49.2, C58.2, C71.2, C8.1, CARD1.4 (VDD), D9.2 (VDD), JP7.3 (B), L1.2, L4.2, Q1.2 (S), R14.1, R16.1, R17.1, R18.1, R29.1, R30.1, R31.1, R32.1, R38.2, R39.2, R8.1, TP7.1, U11.16 (VDD), U12.8 (VDD), U16.5 (VDD), U7.2 (VDD3P3), U7.20 (VDD3P3_RTC), U7.3 (VDD3P3), U7.55 (VDDA), U7.56 (VDDA), U8.2 (VDD3P3), U8.20 (VDD3P3_RTC), U8.3 (VDD3P3), U8.55 (VDDA), U8.56 (VDDA)
- net +3V3_RF: now also TST-R5.1; no longer L2.1, TP3.1
- net 2CHIP_BOOT: now also C69.2
- net 2CHIP_PU: now also C57.2, R52.1, RST2.2; no longer PB1.2
- net 2GPIO1: now also TP4.1
- net 2GPIO14: now also TP9.1
- net 2GPIO2: now also TP5.1; no longer C45.2, R38.1, U11.18 (CLK)
- net 2GPIO26: now also TP17.1
- net 2GPIO3: now also TP6.1; no longer C47.2, R39.1, U11.17 (DIO)
- net 2GPIO33: now also TP20.1
- net 2GPIO34: now also TP21.1
- net 2GPIO35: now also TP22.1
- net 2GPIO36: now also TP23.1
- net 2GPIO37: now also TP24.1
- net 2GPIO38: now also TP25.1
- net 2GPIO39: now also TP26.1
- net 2GPIO40: now also TP27.1
- net 2GPIO41: now also TP28.1
- net 2GPIO42: now also TP29.1
- net 2GPIO45: now also TP30.1
- net 2GPIO46: now also TP31.1
- net 2GPIO47: now also TP19.1
- net 2GPIO48: now also TP18.1
- net 2GPIO7: now also TP7.1
- net 2GPIO8: now also TP8.1
- net CAM.D0: now also FPC1.19 (19_Y2-D0)
- net CAM.D1: no longer FPC1.19 (19_Y2-D0)
- net Earth: now also C26.1, C28.2, C29.2, C31.2, C32.2, JP7.3 (B), C2.2, C23.1, C24.2, C25.2, C27.2, C30.2, C41.1, C42.2, C57.1, C69.1, C72.1, J2.A1 (GND), J2.A12 (GND), J2.B1 (GND), J2.B12 (GND), J2.S1 (SHIELD), JP8.1 (A), R5.2, R7.2, RST2.1, U10.4 (GND), U17.3 (GND), U4.2 (GND); no longer C26.2, C28.1, C29.1, C31.1, C32.1, JP7.1 (A), PB1.1
- net GPIO26: now also TP16.1
- net ISEN.FLT: now also C2.1
- net RC.PWR: now also U8.14 (GPIO9)
- net RF2: now also U8.1 (LNA_IN), TP32.1
- net VBUS: now also U2.3 (IP-), U2.4 (IP-), D2.1, TST-R24.2, TST-R3.1, TST-R4.1; no longer C54.1, C55.1, D11.1, JP3.1 (A), Q2.2 (S), Q3.2 (S), Q4.2 (S), Q5.2 (S), R40.1, R42.1, R43.1, R54.1, R55.1, R56.1, U15.7 (VDD), U15.8 (VDD), U2.1 (IP+), U2.2 (IP+), U3.5 (VBUS)
- net VDD_SPI: no longer U8.29 (VDD_SPI)
- net Vdrive: now also JP3.1 (A), R40.1, U2.1 (IP+), U2.2 (IP+), TST-R1.1, TST-R16.1, TST-R17.2, TST-R18.2, TST-R21.2, TST-R22.2, TST-R23.1; no longer C1.1, R3.1, TP1.1, U1.4 (VIN), U2.3 (IP-), U2.4 (IP-)
- net 7SEG.K2: now reaches U11.20 (K2)
- net 7SEG.K2: now also PB2.2
- net 2FLASH_QSPI_nCS: now reaches TP44.1
- net 2FLASH_QSPI_nCS: now also R33.1, U10.1 (CS#); no longer U11.19 (K1)
- net at TP15.1: now also FPC1.25
- net at TP14.1: now also FPC1.26
- net at D5.2 (-), D7.2, U14.7 (VIN-)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: now also D6.2 (-)
- net 7SEG.SEG5: now reaches DISP1.1 (E), U11.6 (SEG5/KS5)
- net 7SEG.SEG6: now reaches DISP1.10 (F), U11.7 (SEG6/KS6)
- net 7SEG.GRID1: now reaches DISP1.12 (DIG1), U11.15 (GRID1)
- net 7SEG.SEG7: now reaches DISP1.2 (G), U11.8 (SEG7/KS7)
- net 7SEG.SEG4: now reaches DISP1.3 (D), U11.5 (SEG4/KS4)
- net 7SEG.SEG3: now reaches DISP1.4 (C), U11.4 (SEG3/KS3)
- net 7SEG.SEG2: now reaches DISP1.5 (B), U11.3 (SEG2/KS2)
- net 7SEG.SEG8: now reaches DISP1.6 (DP), U11.9 (SEG8/KS8)
- net 7SEG.GRID3: now reaches DISP1.7 (DIG3), U11.13 (GRID3)
- net 7SEG.GRID2: now reaches DISP1.8 (DIG2), U11.14 (GRID2)
- net 7SEG.SEG1: now reaches DISP1.9 (A), U11.2 (SEG1/KS1)
- net 7SEG.SEG1: now also PB1.1, PB2.1
- net 2GPIO10 renamed RC.PAN
- net RC.PAN: now also J5.1 (Pin_1); no longer J6.1 (Pin_1)
- net 2GPIO11 renamed RC.ROT
- net RC.ROT: now also U8.17 (GPIO12); no longer U8.16 (GPIO11)
- net 2GPIO12 renamed RC.OTHR
- net RC.OTHR: no longer U8.17 (GPIO12)
- net 2GPIO15 renamed 2OSC32_IN
- net 2GPIO16 renamed 2OSC32_OUT
- net 2GPIO17 renamed ISEN.VO
- net 2GPIO18 renamed TEMP.DQ
- net TEMP.DQ: now also U12.1 (DQ)
- net 2GPIO19 renamed 2USB_D-
- net 2USB_D-: now also R12.2, U4.1 (I/O1), U4.6 (I/O1)
- net 2GPIO20 renamed 2USB_D+
- net 2USB_D+: now also R13.2, U4.3 (I/O2), U4.4 (I/O2)
- net 2GPIO27 renamed 2FLASH_QSPI_nH
- net 2FLASH_QSPI_nH: now also U10.7 (IO3)
- net 2GPIO28 renamed 2FLASH_QSPI_nWP
- net 2FLASH_QSPI_nWP: now also U10.3 (IO2)
- net 2GPIO30 renamed 2FLASH_QSPI_CLK
- net 2FLASH_QSPI_CLK: now also U10.6 (CLK)
- net 2GPIO31 renamed 2FLASH_QSPI_DO
- net 2FLASH_QSPI_DO: now also U10.2 (DO)
- net 2GPIO32 renamed 2FLASH_QSPI_DI
- net 2FLASH_QSPI_DI: now also U10.5 (DI)
- net 2GPIO4 renamed LED.WH
- net 2GPIO43 renamed 2U0TXD
- net 2GPIO44 renamed 2U0RXD
- net 2GPIO5 renamed LED.IR
- net 2GPIO6 renamed LED.OTH
- removed net 2GPIO9: J5.1 (Pin_1), U8.14 (GPIO9)
- net GPIO15 renamed 7SEG.CLK
- net 7SEG.CLK: now also C45.2, R38.1, U11.18 (CLK)
- net GPIO16 renamed 7SEG.DIO
- net 7SEG.DIO: now also C47.2, R39.1, U11.17 (DIO)
- net GPIO19 renamed USB_D-
- net GPIO20 renamed USB_D+
- net GPIO21 renamed SPK.LRCLK
- net GPIO33 renamed MIC.WS
- net MIC.WS: now also U17.1 (WS); no longer U12.1 (DQ)
- net GPIO34 renamed MIC.SD
- net MIC.SD: now also U17.6 (SD)
- net GPIO35 renamed MIC.SCK
- net MIC.SCK: now also U17.4 (SCK)
- net GPIO36 renamed SPK.DIN
- net GPIO37 renamed SPK.BCLK
- net GPIO4 renamed SD.CS
- net GPIO43 renamed U0TXD
- net GPIO44 renamed U0RXD
- net GPIO5 renamed SD.MISO
- net GPIO6 renamed SD.MOSI
- net GPIO7 renamed SD.CLK
- net MIC.LR renamed MIC.R
- new net: C23.2, C24.1, C25.1, C27.1, C30.1, TST-R10.1, U7.2 (VDD3P3), U7.20 (VDD3P3_RTC), U7.3 (VDD3P3), U7.55 (VDDA), U7.56 (VDDA)
- new net: C43.2, C44.1, R38.2, R39.2, TST-R14.1, U11.16 (VDD)
- new net: C8.1, L1.2, R8.1, TST-R2.1
- new net: Q2.2 (S), R42.1, TST-R17.1
- new net: Q1.2 (S), R14.1, TST-R6.1
- new net: D11.1, TST-R24.1
- new net: C54.1, C55.1, TST-R18.1, U15.7 (VDD), U15.8 (VDD)
- new net: D2.2, J2.A4 (VBUS), J2.A9 (VBUS), J2.B4 (VBUS), J2.B9 (VBUS)
- new net: Q3.2 (S), R54.1, TST-R21.1
- new net: C1.1, R3.1, TP1.1, TST-R1.2, U1.4 (VIN)
- new net: C17.1, C19.2, TST-R8.1, U5.2 (VO)
- new net: C35.2, L4.2, TST-R12.1
- new net: C72.2, TST-R26.1, U17.5 (VDD)
- new net: R16.1, R17.1, R18.1, TST-R7.2
- new net: C26.2, C28.1, C29.1, C31.1, C32.1, TST-R11.1, U8.2 (VDD3P3), U8.20 (VDD3P3_RTC), U8.3 (VDD3P3), U8.55 (VDDA), U8.56 (VDDA)
- new net: C38.2, CARD1.4 (VDD), R29.1, R30.1, R31.1, R32.1, TST-R13.1
- new net: JP8.3 (B), TST-R27.1
- new net: TST-R3.2, U3.5 (VBUS)
- new net: C18.1, C20.2, TST-R9.1, U6.2 (VO)
- new net: R43.1, TST-R16.2
- new net: C71.2, TST-R25.1, U16.5 (VDD)
- new net: Q5.2 (S), R56.1, TST-R23.2
- new net: JP7.1 (A), TST-R20.1
- new net: L2.1, TP3.1, TST-R5.2
- new net: C58.2, D9.2 (VDD), TST-R19.1
- new net: TST-R4.2, U4.5 (VBUS)
- new net: C49.2, TST-R15.2, U12.8 (VDD)
- new net: Q4.2 (S), R55.1, TST-R22.1
- new net 2USB_CC1: J2.A5 (CC1), R7.1
- new net 2USB_CC2: J2.B5 (CC2), R5.1
- new net 2USB_PRT_D+: J2.A6 (D+), J2.B6 (D+), R13.1
- new net 2USB_PRT_D-: J2.A7 (D-), J2.B7 (D-), R12.1
- new net 2VDD_SPI: C41.2, C42.1, R33.2, TP49.1, U10.8 (VCC), U8.29 (VDD_SPI)
- new net 7SEG.K1: PB1.2, U11.19 (K1)
- new net MIC.L: JP8.2 (C), U17.2 (LR)
- new net RC.TILT: J6.1 (Pin_1), U8.16 (GPIO11)
- no-connect marks 9 -> 11
Other:
- note added: "2GPIO10"
- note added: "2GPIO11"
- note added: "2GPIO12"
- note added: "2GPIO13"
- note added: "2GPIO15"
- note added: "2GPIO16"
- note added: "2GPIO17"
- note added: "2GPIO18"
- note added: "2GPIO19"
- note added: "2GPIO20"
- note added: "2GPIO21"
- note added: "2GPIO27"
- note added: "2GPIO28"
- note added: "2GPIO29"
- note added: "2GPIO30"
- note added: "2GPIO31"
- note added: "2GPIO32"
- note added: "2GPIO4"
- note added: "2GPIO43"
- note added: "2GPIO44"
- note added: "2GPIO5"
- note added: "2GPIO6"
- note added: "2GPIO9"
- note added: "2USB_C"
- note added: "Current Sense"
- note added: "FC = 1/(2*PI*Rfint*Cfilter) 88Hz = 1/(2*PI*1.8kohm*1nF)"
- note added: "GPIO1"
- note added: "GPIO10"
- note added: "GPIO11"
- note added: "GPIO12"
- note added: "GPIO13"
- note added: "GPIO14"
- note added: "GPIO15"
- note added: "GPIO16"
- note added: "GPIO17"
- note added: "GPIO18"
- note added: "GPIO19"
- note added: "GPIO2"
- note added: "GPIO20"
- note added: "GPIO21"
- note added: "GPIO27"
- note added: "GPIO28"
- note added: "GPIO29"
- note added: "GPIO3"
- note added: "GPIO30"
- note added: "GPIO31"
- note added: "GPIO32"
- note added: "GPIO33"
- note added: "GPIO34"
- note added: "GPIO35"
- note added: "GPIO36"
- note added: "GPIO37"
- note added: "GPIO38"
- note added: "GPIO39"
- note added: "GPIO4"
- note added: "GPIO40"
- note added: "GPIO41"
- note added: "GPIO42"
- note added: "GPIO43"
- note added: "GPIO44"
- note added: "GPIO45"
- note added: "GPIO46"
- note added: "GPIO47"
- note added: "GPIO48"
- note added: "GPIO5"
- note added: "GPIO6"
- note added: "GPIO7"
- note added: "GPIO8"
- note added: "GPIO9"
- note added: "I2S CHANNEL LR = HI = RIGHT LR = LOW = LEFT"
- note added: "LIGHTS"
- note added: "MICROPHONES"
- note added: "PCB TEMPERATURE"
- note added: "TODO MAKE SURE ALL COMPONENTS CAN BE SOURCED LIKE L2, L4"
- note removed: "Decoupling Capacitors (MCU)"
- note removed: "Imax = 200mA"
- note removed: "MICROPHONE"
- note removed: "TEMPERATURE"
- note removed: "WS2812-2020"
- moved on the sheet: ANT1, BOOT1, C1, C10, C11, C12, C13, C14, C15, C16, C17, C18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

Commit message: draft commit
Parts:
- removed BOOT1, BOOT2: SW_BOOT, Button_Switch_SMD:SW_SPST_EVQP2, symbol Switch:SW_Push
- removed J1, J2: USB-C, Connector_USB:USB_C_Receptacle_GCT_USB4105-xx-A_16P_TopMnt_Horizontal, symbol PCB_Lib_DaanHeetkamp:USB_C_Receptacle_USB2.0
- removed PB1, PB2, RST1, RST2: SW_RST, Button_Switch_SMD:SW_SPST_EVQP2, symbol Switch:SW_Push
- added BOOT1, BOOT2, PB1, PB2, RST2, RST3: Tactile Button, 160gf, PCM_JLCPCB:SW-SMD_4P-L5.1-W5.1-P3.70-LS6.5-TL-2, symbol PCM_JLCPCB-Connectors_Buttons:Tactile Button, 160gf
- added J1, J2: Connector, USB-TYPE-C-16P, PCM_JLCPCB:TYPE-C-SMD_HX-TYPE-C-16PIN, symbol PCM_JLCPCB-Extended:Connector, USB-TYPE-C-16P
- J10, J11, J12, J13, J3, J4, J5, J6, J7, J8, JP3, JP4, JP5, JP6, JP7, JP8: now not fitted
- L1: value 2u2 -> 2.2uH; Manufacturer_Name SXN(Shun Xiang Nuo Elec) -> (none); Manufacturer_Part_Number SMNR4020-2.2UH -> (none)
- L2, L3: value 2n2 -> 2nH; Manufacturer_Name Sunlord -> (none); Manufacturer_Part_Number SDCL1608C2N2STDF -> (none)
- R8: Manufacturer_Name FOJAN -> (none); Manufacturer_Part_Number FRC0402F4503TS -> (none)
- U10, U13: value W25Q128 -> W25Q128JVSIQ
- U6: Attrition Qty 2 -> (none); Category Power Management ICs,Linear Voltage Regulators (LDO) -> (none); Class Basic Component -> (none); Dropout Voltage 680mV@(100mA) -> (none); Feature Low ESR;Overcurrent Protection(OCP) -> (none); LCSC C2892669 -> C41424780; Manufacturer Torex Semicon -> (none); Maximum Input Voltage 6V -> (none); Minimum Qty 5 -> (none); Number Of Outputs 1 -> (none); Output Current 200mA -> (none); Output Polarity Positive electrode -> (none); Output Type Fixed -> (none); Output Voltage 3.3V -> (none); Part XC6206P332MR-G -> (none); Price 0.103USD -> (none); Process SMT -> (none); Stock 310885 -> (none)
- Y1, Y2: LCSC PART # C2885592 -> C9010; Manufacturer_Name YXC Crystal Oscillators -> (none); Manufacturer_Part_Number X252040MMB4SI -> (none); Name X252040MMB4SI -> (none)
- Y3: LCSC PART # C93232 -> C97604
- renumbered C70 to C68, C71 to C69, C72 to C70, C68 to C71, C69 to C72, R6 to R5, R5 to R6, TP11 to TP10, TP12 to TP11, TP13 to TP12, TP14 to TP13, TP15 to TP14, TP16 to TP15, TP17 to TP16, TP18 to TP17, TP19 to TP18, TP20 to TP19, TP21 to TP20, TP22 to TP21, TP23 to TP22, TP24 to TP23, TP25 to TP24, TP26 to TP25, TP27 to TP26, TP28 to TP27, TP29 to TP28, TP30 to TP29, TP31 to TP30, TP32 to TP31, TP33 to TP32, TP34 to TP33, TP35 to TP34, TP36 to TP35, TP37 to TP36, TP38 to TP37, TP39 to TP38, TP40 to TP39, TP41 to TP40, TP42 to TP41, TP43 to TP42, TP44 to TP43, TP45 to TP44, TP46 to TP45, TP47 to TP46, TP48 to TP47, TP49 to TP48, TP50 to TP49, TP51 to TP50, TP52 to TP51, TP53 to TP52, TP54 to TP53, TP55 to TP54, TP56 to TP55, TP57 to TP56, TP58 to TP57, TP59 to TP58, TP60 to TP59, TP61 to TP60, TP62 to TP61, TP63 to TP62, TP64 to TP63, TP65 to TP64, TP66 to TP65, TP67 to TP66, TP68 to TP67, TST-R27 to TST-R21, TST-R21 to TST-R22, TST-R22 to TST-R23, TST-R23 to TST-R24, TST-R24 to TST-R25, TST-R25 to TST-R26, TST-R26 to TST-R27
Connections:
- net 2CHIP_BOOT: now also BOOT2.1 (A)
- net 2CHIP_PU: now also RST3.1 (A)
- net 2USB_CC1: now also R6.1, J2.A5 (CC1); no longer R7.1
- net 2USB_CC2: now also R7.1, J2.B5 (CC2); no longer R6.1
- net 2USB_PRT_D+: now also J2.A6 (D+), J2.B6 (D+)
- net 2USB_PRT_D-: now also J2.A7 (D-), J2.B7 (D-)
- net 7SEG.K1: now also PB1.2 (B)
- net 7SEG.K2: now also PB2.2 (B)
- net 7SEG.SEG1: now also PB1.4 (D), PB2.4 (D)
- net CHIP_BOOT: now also BOOT1.1 (A)
- net CHIP_PU: now also RST2.1 (A)
- net Earth: now also BOOT1.3 (C), BOOT2.3 (C), J1.A12B1 (GND), J1.B12A1 (GND), J1.S1 (SHIELD), J2.A12B1 (GND), J2.B12A1 (GND), J2.S1 (SHIELD), RST2.3 (C), RST3.3 (C)
- net USB_CC1: now also R4.1, J1.A5 (CC1); no longer R5.1
- net USB_CC2: now also R5.1, J1.B5 (CC2); no longer R4.1
- net USB_PRT_D+: now also J1.A6 (D+), J1.B6 (D+)
- net USB_PRT_D-: now also J1.A7 (D-), J1.B7 (D-)
- net at D2.2: now also J2.A9B4 (VBUS), J2.B9A4 (VBUS)
- net at D1.2: now also J1.A9B4 (VBUS), J1.B9A4 (VBUS)
- no-connect marks 11 -> 23
Other:
- note added: "expected risky area -- camera connector pinout, is pin1 really pin 1 not 24? -- I2S microphones and amplifier, should they be the same lines like code suggests -- I2C, does this need pull up, or can internal pullup suffice? -- POE ethernet, complete unknown. Fingers crossed. TODO -- MAKE SURE ALL COMPONENTS CAN BE SOURCED LIKE L2, L4 -- add dip switches to specify room number -- make office conso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"
- note removed: "TODO MAKE SURE ALL COMPONENTS CAN BE SOURCED LIKE L2, L4"
- moved on the sheet: C56, C57, C71, C72, R4, R5, R6, R7

Commit message: draft commit
Parts:
- removed Y1, Y2: 40MHz, Crystal:Crystal_SMD_3225-4Pin_3.2x2.5mm, symbol Device:Crystal_GND24
- added Y1, Y2: 40MHz, 15pF, JLCPCB:OSC-SMD_4P-L3.2-W2.5-BL_SIT8008BI, symbol JLCPCB-Extended:Crystal, 40MHz, 15pF
- R8: value 450k -> 450kΩ
Connections:
- net 2OSC_OUT: now also Y2.3 (OSC)
- net Earth: now also Y1.2 (GND), Y1.4 (GND), Y2.2 (GND), Y2.4 (GND)
- net OSC_OUT: now also Y1.3 (OSC)
- net at C3.1, R1.1: now also Y1.1 (OSC)
- net at C4.1, R2.1: now also Y2.1 (OSC)
Other:
- moved on the sheet: C3, C6, C7, R1
