File: ESP32S3_Audio_Cam_POE.kicad_sch (KiCad schematic)
At the start: 306 parts, among them J1 Connector, USB-TYPE-C-16P, J10 Conn_01x02, J11 Conn_01x02, J12 Conn_01x02, J13 Conn_01x02, J2 Connector, USB-TYPE-C-16P, J3 Conn_01x02, J4 Conn_01x02, J5 Conn_01x03, J6 Conn_01x03, J7 Conn_01x03, J8 Conn_01x03, J9 HC-RJ45-055-4_8P8C_Shielded, Q1 AO3401A, Q2 AO3401A, Q3 AO3401A, Q4 AO3401A, Q5 AO3401A, T1 H1102NLT, U1 TLV62568DBVR, U10 W25Q128JVSIQ, U11 TM1637, U12 DS18B20U(UMW), U13 W25Q128JVSIQ, U14 DP9900M-5V, U15 MAX98357AETE+T, U16 ICS-43434, U17 ICS-43434, U2 MT9221CT-06BR5, U3 USBLC6-2SC6, U4 USBLC6-2SC6, U5 XC6206-1.5NR, U6 XC6206-2.8V, U7 ESP32-S3, U8 ESP32-S3, U9 W5500, X1 X322525MOB4SI, Y1 40MHz, 15pF, Y2 40MHz, 15pF, Y3 32.768KHz

Commit message: DRAFT added AXP2101 battery circuit
Parts:
- added C73, C88, C90, C91, C92, C93, C94: 1uF, PCM_JLCPCB:C_0402, symbol JLCPCB-Capacitors:0402,1uF
- added C74: 10uF, PCM_JLCPCB:C_0402, symbol JLCPCB-Capacitors:0402,10uF
- added C75, C76, C77, C78, C95: 22uF, PCM_JLCPCB:C_0603, symbol JLCPCB-Capacitors:0603,22uF
- added C79, C80, C81, C82, C83, C84, C85, C86, C87, C96: 2.2uF, PCM_JLCPCB:C_0402, symbol JLCPCB-Capacitors:0402,2.2uF
- added C89: 4.7uF, PCM_JLCPCB:C_0402, symbol JLCPCB-Capacitors:0402,4.7uF
- added D14: Yellow, PCM_JLCPCB:D_0805, symbol JLCPCB-Diodes:LED,0805,Yellow
- added J14, J15, J16: Conn_01x02, Connector_PinHeader_1.00mm:PinHeader_1x02_P1.00mm_Vertical, symbol Connector_Generic:Conn_01x02
- added L5, L6, L7, L8, L9: 1uH,50mA, PCM_JLCPCB:L_0805, symbol JLCPCB-Inductors:1uH,50mA
- added PB3: Tactile Button, 160gf, PCM_JLCPCB:SW-SMD_4P-L5.1-W5.1-P3.70-LS6.5-TL-2, symbol PCM_JLCPCB-Connectors_Buttons:Tactile Button, 160gf
- added R66: 10kΩ, PCM_JLCPCB:R_0402, symbol PCM_JLCPCB-Resistors:0402,10kΩ
- added U18: AXP2101, Package_DFN_QFN:QFN-40-1EP_5x5mm_P0.4mm_EP3.6x3.6mm_ThermalVias, symbol JLCPCB-Extended:AXP2101_C3036461
Connections:
- net Earth: now also C73.1, C74.2, C75.1, C76.1, C77.1, C78.1, C79.1, C80.1, C81.1, C82.1, C83.1, C84.1, C85.1, C86.1, C87.1, C88.1, C89.1, C90.1, C91.1, C92.1, C93.1, C94.1, C95.1, C96.1, J14.2 (Pin_2), J15.2 (Pin_2), J16.2 (Pin_2), PB3.3 (C), U18.3 (GND), U18.41 (EP)
- net VBUS: now also C74.1, C88.2, C89.2, C91.2, C92.2, C93.2, C94.2, R66.2, U18.13 (BLDOIN), U18.17 (ALDOIN), U18.23 (VIN1), U18.24 (VIN2), U18.34 (VSYS), U18.36 (VMID), U18.37 (VBUS), U18.6 (VIN3), U18.7 (VIN4)
- new net: C81.2, U18.15 (ALDO4)
- new net: C86.2, U18.10 (CPULDOS)
- new net: D14.2, R66.1
- new net: D14.1, U18.1 (CHGLED)
- new net: C87.2, U18.11 (DLDO2/DC4SW)
- new net: C84.2, U18.12 (BLDO1)
- new net: C85.2, U18.14 (BLDO2)
- new net: C80.2, U18.16 (ALDO3)
- new net: C79.2, U18.18 (ALDO1)
- new net: C82.2, U18.19 (ALDO2)
- new net: C73.2, U18.2 (VREF)
- new net: C83.2, U18.20 (DLDO1/DC1SW)
- new net: L8.2, U18.21 (FB1)
- new net: C78.2, L8.1, U18.22 (LX1)
- new net: L7.2, U18.25 (LX2)
- new net: C77.2, L7.1, U18.26 (FB2)
- new net: J15.1 (Pin_1), U18.27 (VBACKUP)
- new net: C90.2, U18.28 (VRTC)
- new net: PB3.1 (A), U18.30 (PWRON)
- new net: J16.1 (Pin_1), U18.31 (TS)
- new net: C96.2, J14.1 (Pin_1), U18.33 (BAT)
- new net: L9.2, U18.35 (SW)
- new net: C75.2, L5.1, U18.4 (FB3)
- new net: L5.2, U18.5 (LX3)
- new net: C76.2, L6.1, U18.8 (LX4)
- new net: L6.2, U18.9 (FB4)
- new net VDCDC5: C95.2, L9.1, U18.32 (GPIO1/FB5/RTC/LDO2)
- no-connect marks 23 -> 25

Commit message: DRAFT added AXP2101 battery circuit
Parts:
- added D15: Green, PCM_JLCPCB:D_0805, symbol PCM_JLCPCB-Diodes:LED,0805,Green
- added R67: 10kΩ, PCM_JLCPCB:R_0402, symbol PCM_JLCPCB-Resistors:0402,10kΩ
- added TP68: TestPoint, TestPoint:TestPoint_Pad_D1.0mm, symbol Connector:TestPoint
- L5, L6, L7, L8, L9: value 1uH,50mA -> 1uH,3.3A; footprint PCM_JLCPCB:L_0805 -> Inductor_SMD:L_1008_2520Metric; LCSC C1042 -> C435392
Connections:
- net 2GPIO37 is gone; now on net BAT.SCK: TP23.1, U8.42 (GPIO37)
- net 2GPIO38 is gone; now on net BAT.SDA: TP24.1, U8.43 (GPIO38)
- net VBUS: now also R67.2
- net at U18.29 (PWROK): now also D15.1
- net at U18.38 (IRQ): now also TP68.1
- net BAT.SCK: now reaches U18.39 (SCK)
- net BAT.SDA: now reaches U18.40 (SDA)
- new net: D15.2, R67.1
Other:
- note added: "2GPIO37"
- note added: "2GPIO38"
- note added: "BATTERY PMU / GUAGE"
- moved on the sheet: C73, C74, C75, C76, C77, C78, C79, C80, C81, C82, C83, C84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

Commit message: DRAFT added misc outputs, PMU and resolved some TODO notes.
Parts:
- removed R8: 450kΩ, Resistor_SMD:R_0402_1005Metric_Pad0.72x0.64mm_HandSolder, symbol Device:R
- added BT1: BH-18650-B1BA002, JLCPCB:BATTERY-SMD_18650-1S-L77.1-W20.7-1, symbol JLCPCB-Extended:BH-18650-B1BA002_18650_C2988620
- added C97: 22uF, PCM_JLCPCB:C_0603, symbol JLCPCB-Capacitors:0603,22uF
- added D16, D17, D18: IR, JLCPCB:IR-LED_C131280, symbol JLCPCB-Diodes:LED IR IR26-21c_C131280
- added J17, J18, J19: Conn_01x02, Connector_PinHeader_1.00mm:PinHeader_1x02_P1.00mm_Vertical, symbol Connector_Generic:Conn_01x02
- added NTC1: NTC, PCM_JLCPCB:R_0402, symbol JLCPCB-Resistors:0402,10kΩ
- added PB4, PB5: Tactile Button, 160gf, PCM_JLCPCB:SW-SMD_4P-L5.1-W5.1-P3.70-LS6.5-TL-2, symbol PCM_JLCPCB-Connectors_Buttons:Tactile Button, 160gf
- added Q6, Q7, Q8: AO3401A, PCM_JLCPCB:Q_SOT-23, symbol PCM_JLCPCB-Transistors:PMOS,AO3401A
- added R68, R71, R72: 100kΩ, PCM_JLCPCB:R_0402, symbol PCM_JLCPCB-Resistors:0402,100kΩ
- added R69, R70, R73, R78, R81, R84: 10kΩ, PCM_JLCPCB:R_0402, symbol PCM_JLCPCB-Resistors:0402,10kΩ
- added R74, R76: 220kΩ, PCM_JLCPCB:R_0402, symbol JLCPCB-Resistors:0402,220kΩ
- added R75: 10kΩ, PCM_JLCPCB:R_0402, symbol JLCPCB-Resistors:0402,10kΩ
- added R77, R80, R83: 1MΩ, PCM_JLCPCB:R_0402, symbol PCM_JLCPCB-Resistors:0402,1MΩ
- added R79, R8, R82: 10MΩ, PCM_JLCPCB:R_0402, symbol PCM_JLCPCB-Resistors:0402,10MΩ
- added TP69, TP70, TP71, TP72, TP73, TP74, TP75, TP76, TP77, TP78, TP79, TP80, TP81, TP82, TP83, TP84: TestPoint, TestPoint:TestPoint_Loop_D3.50mm_Drill0.9mm_Beaded, symbol Connector:TestPoint
- added TST-R28, TST-R29, TST-R30, TST-R31, TST-R32: 0Ω, PCM_JLCPCB:R_0603, symbol PCM_JLCPCB-Resistors:0603,0Ω
Connections:
- net 2GPIO26 is gone; now on net PMU.Vref: TP16.1, U8.28 (SPICS1)
- net +3V3: now also R72.2, TST-R29.2
- net 7SEG.K1: now also PB4.2 (B)
- net 7SEG.K2: now also PB5.2 (B)
- net 7SEG.SEG2: now also PB5.4 (D)
- net 7SEG.SEG3: now also PB4.4 (D)
- net Earth: now also BT1.1, C97.1, D16.1 (C), D17.1 (C), D18.1 (C), J17.2 (Pin_2), J18.2 (Pin_2), J19.2 (Pin_2), NTC1.1, R69.2, R70.2, R73.2
- net VBUS: now also R68.2; no longer C74.1, C88.2, C89.2, C91.2, C92.2, C93.2, C94.2, R66.2, R67.2, U18.13 (BLDOIN), U18.17 (ALDOIN), U18.23 (VIN1), U18.24 (VIN2), U18.34 (VSYS), U18.36 (VMID), U18.37 (VBUS), U18.6 (VIN3), U18.7 (VIN4)
- net VDCDC5: now also C97.2, TP84.1
- net Vdrive: now also TST-R28.2, TST-R30.2, TST-R31.2, TST-R32.2
- net PMU.Va4: now reaches C81.2, U18.15 (ALDO4)
- net PMU.Va4: now also TP80.1
- net at C8.1, L1.2, TST-R2.1: now also R76.1
- net PMU.Vcpu: now reaches C86.2, U18.10 (CPULDOS)
- net PMU.Vcpu: now also TP82.1
- net at R9.1, U1.5 (FB): now also R75.2
- net PMU.Vd2: now reaches C87.2, U18.11 (DLDO2/DC4SW)
- net PMU.Vd2: now also TP76.1
- net PMU.Vb1: now reaches C84.2, U18.12 (BLDO1)
- net PMU.Vb1: now also TP73.1
- net PMU.Vb2: now reaches C85.2, U18.14 (BLDO2)
- net PMU.Vb2: now also TP74.1
- net PMU.Va3: now reaches C80.2, U18.16 (ALDO3)
- net PMU.Va3: now also TP79.1
- net PMU.Va1: now reaches C79.2, U18.18 (ALDO1)
- net PMU.Va1: now also TP77.1
- net PMU.Va2: now reaches C82.2, U18.19 (ALDO2)
- net PMU.Va2: now also TP78.1
- net PMU.Vref: now reaches C73.2, U18.2 (VREF)
- net PMU.Vref: now also TP83.1
- net PMU.Vd1: now reaches C83.2, U18.20 (DLDO1/DC1SW)
- net PMU.Vd1: now also TP75.1
- net PMU.Vo1: now reaches C78.2, L8.1, U18.22 (LX1)
- net PMU.Vo1: now also R71.2, TP69.1, TST-R29.1
- net PMU.Vo2: now reaches C77.2, L7.1, U18.26 (FB2)
- net PMU.Vo2: now also TP70.1
- net at J16.1 (Pin_1), U18.31 (TS): now also NTC1.2
- net at C96.2, J14.1 (Pin_1), U18.33 (BAT): now also BT1.2
- net PMU.Vo3: now reaches C75.2, L5.1, U18.4 (FB3)
- net PMU.Vo3: now also TP71.1
- net PMU.Vo4: now reaches C76.2, L6.1, U18.8 (LX4)
- net PMU.Vo4: now also TP72.1
- net 2GPIO14 renamed VBus.Sense
- net VBus.Sense: now also R68.1, R69.1
- net 2GPIO2 renamed 3v3.Sense
- net 3v3.Sense: now also R72.1, R73.1
- net 2GPIO33 renamed PMU.Vo1.Sense
- net PMU.Vo1.Sense: now also R70.1, R71.1
- net 2GPIO34 renamed MISC.OUT1
- net MISC.OUT1: now also R77.2
- net 2GPIO35 renamed MISC.OUT2
- net MISC.OUT2: now also R80.2
- net 2GPIO36 renamed MISC.OUT3
- net MISC.OUT3: now also R83.2
- net BAT.SCK renamed PMU.SCK
- net BAT.SDA renamed PMU.SDA
- new net: Q7.2 (S), R79.1, TST-R31.1
- new net: Q7.1 (G), R79.2, R80.1
- new net: J17.1 (Pin_1), Q6.3 (D), R78.1
- new net: Q8.1 (G), R82.2, R83.1
- new net: Q6.1 (G), R77.1, R8.2
- new net: C74.1, TST-R28.1, U18.37 (VBUS)
- new net: R74.2, R76.2
- new net: R74.1, R75.1
- new net: D16.2 (A), R78.2
- new net: Q6.2 (S), R8.1, TST-R30.1
- new net: J19.1 (Pin_1), Q8.3 (D), R84.1
- new net: D18.2 (A), R84.2
- new net: J18.1 (Pin_1), Q7.3 (D), R81.1
- new net: D17.2 (A), R81.2
- new net: Q8.2 (S), R82.1, TST-R32.1
- new net PMU.Vsys: C88.2, C89.2, C91.2, C92.2, C93.2, C94.2, R66.2, R67.2, TP81.1, U18.13 (BLDOIN), U18.17 (ALDOIN), U18.23 (VIN1), U18.24 (VIN2), U18.34 (VSYS), U18.36 (VMID), U18.6 (VIN3), U18.7 (VIN4)
- no-connect marks 25 -> 27
Other:
- note added: "2GPIO14"
- note added: "2GPIO2"
- note added: "2GPIO26"
- note added: "2GPIO33"
- note added: "2GPIO34"
- note added: "2GPIO35"
- note added: "2GPIO36"
- note added: "450k equiv"
- note added: "FB is 0.6V, with R9 at 100k, high side wants 450k for 3.3V out."
- note added: "MISC OUTPUTS"
- note added: "NTC wants to be TH11-3H103F while C3018545 is probably a close enough equiv."
- note added: "expected risky area -- camera connector pinout, is pin1 really pin 1 not 24? -- I2S microphones and amplifier, should they be the same lines like code suggests -- I2C, does this need pull up, or can internal pullup suffice? -- POE ethernet, complete unknown. Fingers crossed. TODO -- make office console version, with multiple rooms which can be selected. -- add headphone jack, for quite speaker mo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"
- note removed: "expected risky area -- camera connector pinout, is pin1 really pin 1 not 24? -- I2S microphones and amplifier, should they be the same lines like code suggests -- I2C, does this need pull up, or can internal pullup suffice? -- POE ethernet, complete unknown. Fingers crossed. TODO -- MAKE SURE ALL COMPONENTS CAN BE SOURCED LIKE L2, L4 -- add dip switches to specify room number -- make office conso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"
- moved on the sheet: C1, C43, C44, C45, C47, C73, C79, C8, C80, C81, C82, C83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

Commit message: DRAFT added mic jack.
Parts:
- added CN1: PJ-316C-6A, JLCPCB:SMD_3.5mm_Audio_Connectors_(Headphones)_C707223, symbol JLCPCB-Extended:PJ-316C-6A_SMD_3.5mm_Audio_Connectors_(Headphones)_C707223
- added TP85: TestPoint, TestPoint:TestPoint_Pad_D1.0mm, symbol Connector:TestPoint
Connections:
- net SPK.OutN: now reaches C66.2, U15.10 (OUTN)
- net SPK.OutN: now also J10.2 (Pin_2), CN1.1; no longer J10.1 (Pin_1)
- net SPK.OutP: now reaches C67.1, U15.9 (OUTP)
- net SPK.OutP: now also CN1.2, CN1.3; no longer J10.2 (Pin_2)
- new net SPK.MIC: CN1.4, TP85.1
- new net SPK.OutPS: CN1.5, CN1.6, J10.1 (Pin_1)
Other:
- note added: "expected risky area -- camera connector pinout, is pin1 really pin 1 not 24? -- I2S microphones and amplifier, should they be the same lines like code suggests -- I2C, does this need pull up, or can internal pullup suffice? -- POE ethernet, complete unknown. Fingers crossed. TODO -- make office console version, with multiple rooms which can be selected. -- Make light bar, to be attached to the J1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"
- note removed: "expected risky area -- camera connector pinout, is pin1 really pin 1 not 24? -- I2S microphones and amplifier, should they be the same lines like code suggests -- I2C, does this need pull up, or can internal pullup suffice? -- POE ethernet, complete unknown. Fingers crossed. TODO -- make office console version, with multiple rooms which can be selected. -- add headphone jack, for quite speaker mo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"
- moved on the sheet: C54, C55, C66, C67, J10, JP3, JP4, JP5, JP6, R40, R41, R43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

Commit message: Draft Updated ESP32-S3 now includes 8MB internal PSRAM
Parts:
- U7, U8: LCSC C2913192 -> C2913194

Commit message: Draft Misc changes, layout still needs a lot of work.
Parts:
- added TP100, TP101, TP102, TP103, TP104, TP105, TP106, TP107, TP108, TP109, TP110, TP111, TP112, TP113, TP114, TP115, TP116, TP117, TP118, TP119, TP120, TP121, TP122, TP123, TP124, TP125, TP126, TP127, TP128, TP129, TP86, TP87, TP88, TP89, TP90, TP91, TP92, TP93, TP94, TP95, TP96, TP97, TP98, TP99: TestPoint, Connector_PinHeader_1.00mm:PinHeader_1x01_P1.00mm_Vertical, symbol Connector:TestPoint
- TP69, TP70, TP71, TP72, TP73, TP74, TP75, TP76, TP77, TP78, TP79, TP80, TP81, TP82, TP83, TP84: footprint TestPoint:TestPoint_Loop_D3.50mm_Drill0.9mm_Beaded -> Connector_PinHeader_1.00mm:PinHeader_1x01_P1.00mm_Vertical
Connections:
- net +1V5: now also TP102.1, TP103.1
- net +2V8: now also TP104.1, TP105.1, TP90.1, TP91.1
- net CAM.D0: now also TP120.1, TP121.1
- net CAM.D1: now also TP124.1, TP125.1
- net CAM.D2: now also TP126.1, TP127.1
- net CAM.D3: now also TP122.1, TP123.1
- net CAM.D4: now also TP118.1, TP119.1
- net CAM.D5: now also TP114.1, TP115.1
- net CAM.D6: now also TP110.1, TP111.1
- net CAM.D7: now also TP106.1, TP107.1
- net CAM.HREF: now also TP100.1, TP101.1
- net CAM.MCLK: now also TP108.1, TP109.1
- net CAM.PCLK: now also TP116.1, TP117.1
- net CAM.PWDN: now also TP98.1, TP99.1
- net CAM.RST: now also TP94.1, TP95.1
- net CAM.SCL: now also TP92.1, TP93.1
- net CAM.SDA: now also TP88.1, TP89.1
- net CAM.VSYNC: now also TP96.1, TP97.1
- net Earth: now also TP112.1, TP113.1, TP86.1, TP87.1
- net at FPC1.23 (23_Y1-NC), TP11.1: now also TP128.1, TP129.1
Other:
- moved on the sheet: C16, C17, C18, C19, C20, C21, C22, Q1, R14, R15, R16, R17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
