File: ESP32S3_Audio_Cam_POE_Smaller.kicad_pcb (KiCad board)
At the start: 2 copper layers, 97.5 x 45.7 mm, 52 parts, among them CN1 PJ-316C-6A, J1 Conn_01x20_Pin, J10 Conn_01x02, J2 Conn_01x20_Pin, U11 TM1637, U15 MAX98357AETE+T, U16 ICS-43434, U17 ICS-43434

Commit message: Draft
Parts:
- added ANT1: KH-3216-H0209, JLCPCB:ANT-SMD_L3.2-W1.6-KH-3216F245C04, F.Cu at (32.4, 83.6)
- added BOOT1: Tactile Button, 160gf, PCM_JLCPCB:SW-SMD_4P-L5.1-W5.1-P3.70-LS6.5-TL-2, F.Cu at (47.9, 93.4)
- added BT1: BH-18650-B1BA002, JLCPCB:BATTERY-SMD_18650-1S-L77.1-W20.7-1, B.Cu at (207.4, 116.0)
- added C1: 100nF, PCM_JLCPCB:C_0603, F.Cu at (106.6, 99.8)
- added C10: 10uF, PCM_JLCPCB:C_0402, F.Cu at (96.8, 90.2)
- added C11: 1uF, PCM_JLCPCB:C_0603, F.Cu at (91.3, 49.6)
- added C12: 100nF, PCM_JLCPCB:C_0603, F.Cu at (65.9, 55.0)
- added C13: 100nF, PCM_JLCPCB:C_0603, F.Cu at (94.3, 51.6)
- added C14: 100nF, PCM_JLCPCB:C_0603, F.Cu at (88.3, 48.6)
- added C15: 100nF, PCM_JLCPCB:C_0603, F.Cu at (91.3, 52.6)
- added C16: 100nF, PCM_JLCPCB:C_0603, F.Cu at (48.9, 99.4)
- added C17: 100nF, PCM_JLCPCB:C_0603, F.Cu at (54.9, 91.5)
- added C18: 100nF, PCM_JLCPCB:C_0603, F.Cu at (57.9, 26.1)
- added C19: 3.3pF, PCM_JLCPCB:C_0402, F.Cu at (36.8, 83.4)
- added C2: 1nF, PCM_JLCPCB:C_0402, F.Cu at (118.7, 100.0)
- added C20: 3.3pF, PCM_JLCPCB:C_0402, F.Cu at (37.8, 83.4)
- added C21: 10pF, PCM_JLCPCB:C_0402, F.Cu at (31.5, 57.1)
- added C22: 1uF, PCM_JLCPCB:C_0402, F.Cu at (203.9, 121.1)
- added C23: 10pF, PCM_JLCPCB:C_0402, F.Cu at (34.5, 57.1)
- added C24: 20pF, PCM_JLCPCB:C_0402, F.Cu at (32.7, 59.4)
- added C25: 20pF, PCM_JLCPCB:C_0402, F.Cu at (33.7, 59.4)
- added C26: 10uF, PCM_JLCPCB:C_0402, F.Cu at (199.9, 122.1)
- added C27: 22uF, PCM_JLCPCB:C_0603, F.Cu at (205.9, 125.1)
- added C28: 1uF, PCM_JLCPCB:C_0402, F.Cu at (216.9, 117.1)
- added C29: 22uF, PCM_JLCPCB:C_0603, F.Cu at (201.9, 121.1)
- added C30: 1uF, PCM_JLCPCB:C_0402, F.Cu at (219.9, 117.1)
- added C31: 22uF, PCM_JLCPCB:C_0603, F.Cu at (202.9, 124.1)
- added C32: 2.2uF, PCM_JLCPCB:C_0402, F.Cu at (205.9, 131.1)
- added C33: 22uF, PCM_JLCPCB:C_0603, F.Cu at (208.9, 125.1)
- added C34: 2.2uF, PCM_JLCPCB:C_0402, F.Cu at (206.9, 131.1)
- added C35: 2.2uF, PCM_JLCPCB:C_0402, F.Cu at (210.9, 125.1)
- added C36: 2.2uF, PCM_JLCPCB:C_0402, F.Cu at (210.9, 122.1)
- added C37: 100nF, PCM_JLCPCB:C_0603, F.Cu at (81.1, 22.8)
- added C38: 1uF, PCM_JLCPCB:C_0603, F.Cu at (81.1, 19.8)
- added C39: 4.7uF, PCM_JLCPCB:C_0402, F.Cu at (217.9, 117.1)
- added C40: 1uF, PCM_JLCPCB:C_0402, F.Cu at (215.9, 114.1)
- added C41: 2.2uF, PCM_JLCPCB:C_0402, F.Cu at (211.9, 122.1)
- added C42: 2.2uF, PCM_JLCPCB:C_0402, F.Cu at (209.9, 97.1)
- added C43: 2.2uF, PCM_JLCPCB:C_0402, F.Cu at (216.9, 114.1)
- added C44: 22uF, PCM_JLCPCB:C_0603, F.Cu at (211.9, 109.1)
- added C45: 1uF, PCM_JLCPCB:C_0402, F.Cu at (215.9, 117.1)
- added C46: 1uF, PCM_JLCPCB:C_0402, F.Cu at (218.9, 117.1)
- added C47: 2.2uF, PCM_JLCPCB:C_0402, F.Cu at (214.9, 114.1)
- added C48: 1uF, PCM_JLCPCB:C_0402, F.Cu at (214.9, 117.1)
- added C49: 100nF, PCM_JLCPCB:C_0603, F.Cu at (72.3, 81.1)
- added C50: 2.2uF, PCM_JLCPCB:C_0402, F.Cu at (213.9, 106.1)
- added C51: 2.2uF, PCM_JLCPCB:C_0402, F.Cu at (211.9, 106.1)
- added C52: 22uF, PCM_JLCPCB:C_0603, F.Cu at (212.9, 117.1)
- added C8: 100nF, PCM_JLCPCB:C_0603, F.Cu at (99.4, 89.9)
- added C9: 100nF, PCM_JLCPCB:C_0603, F.Cu at (96.6, 86.0)
- added D1: 1N4148W, PCM_JLCPCB:D_SOD-123, F.Cu at (107.6, 24.7)
- added D2: IR, JLCPCB:IR-LED_C131280, F.Cu at (34.6, 30.8)
- added D3: White, PCM_JLCPCB:D_0603, F.Cu at (134.3, 88.3)
- added D4: WS2812B, PCM_JLCPCB:LED-SMD_4P-L1.6-W1.5_XL-1615RGBC-WS2812B, F.Cu at (56.0, 26.1)
- added D5: IR, JLCPCB:IR-LED_C131280, F.Cu at (30.0, 28.8)
- added D6: IR, JLCPCB:IR-LED_C131280, F.Cu at (124.3, 79.8)
- added D7: Yellow, PCM_JLCPCB:D_0805, F.Cu at (198.9, 116.1)
- added D8: IR, JLCPCB:IR-LED_C131280, F.Cu at (32.6, 23.8)
- added D9: Green, PCM_JLCPCB:D_0805, F.Cu at (198.9, 111.1)
- added J1: Connector, USB-TYPE-C-16P, PCM_JLCPCB:TYPE-C-SMD_HX-TYPE-C-16PIN, F.Cu at (128.7, 26.0)
- added J10: Conn_01x02, Connector_PinHeader_1.00mm:PinHeader_1x02_P1.00mm_Vertical, F.Cu at (135.2, 78.3)
- added J11: Conn_01x03, Connector_PinHeader_2.54mm:PinHeader_1x03_P2.54mm_Vertical, F.Cu at (111.5, 54.8)
- added J12: Conn_01x02, Connector_PinHeader_1.00mm:PinHeader_1x02_P1.00mm_Vertical, F.Cu at (204.9, 128.1)
- added J13: Conn_01x02, Connector_PinHeader_1.00mm:PinHeader_1x02_P1.00mm_Vertical, F.Cu at (206.9, 101.1)
- added J14: Conn_01x03, Connector_PinHeader_2.54mm:PinHeader_1x03_P2.54mm_Vertical, F.Cu at (111.5, 51.0)
- added J15: Conn_01x02, Connector_PinHeader_1.00mm:PinHeader_1x02_P1.00mm_Vertical, F.Cu at (206.9, 98.1)
- added J2: Conn_01x02, Connector_PinHeader_1.00mm:PinHeader_1x02_P1.00mm_Vertical, F.Cu at (35.6, 26.8)
- added J3: Conn_01x02, Connector_PinHeader_1.00mm:PinHeader_1x02_P1.00mm_Vertical, F.Cu at (134.6, 85.0)
- added J4: Conn_01x02, Connector_PinHeader_1.00mm:PinHeader_1x02_P1.00mm_Vertical, F.Cu at (74.3, 63.3)
- added J5: Conn_01x02, Connector_PinHeader_1.00mm:PinHeader_1x02_P1.00mm_Vertical, F.Cu at (38.8, 41.9)
- added J6: Conn_01x02, Connector_PinHeader_1.00mm:PinHeader_1x02_P1.00mm_Vertical, F.Cu at (135.0, 81.6)
- added J7: Conn_01x03, Connector_PinHeader_2.54mm:PinHeader_1x03_P2.54mm_Vertical, F.Cu at (111.4, 62.5)
- added J8: Conn_01x03, Connector_PinHeader_2.54mm:PinHeader_1x03_P2.54mm_Vertical, F.Cu at (111.5, 58.6)
- added J9: Conn_01x02, Connector_PinHeader_1.00mm:PinHeader_1x02_P1.00mm_Vertical, F.Cu at (35.6, 23.8)
- added L3: 2nH, Inductor_SMD:L_0603_1608Metric_Pad1.05x0.95mm_HandSolder, F.Cu at (93.7, 85.8)
- added L4: 2nH, Inductor_SMD:L_0603_1608Metric_Pad1.05x0.95mm_HandSolder, F.Cu at (34.8, 83.4)
- added L5: 1uH,3.3A, Inductor_SMD:L_1008_2520Metric, F.Cu at (205.9, 121.1)
- added L6: 1uH,3.3A, Inductor_SMD:L_1008_2520Metric, F.Cu at (201.9, 117.1)
- added L7: 1uH,3.3A, Inductor_SMD:L_1008_2520Metric, F.Cu at (208.9, 121.1)
- added L8: 1uH,3.3A, Inductor_SMD:L_1008_2520Metric, F.Cu at (201.9, 112.1)
- added L9: 1uH,3.3A, Inductor_SMD:L_1008_2520Metric, F.Cu at (212.9, 113.1)
- added NTC1: NTC, PCM_JLCPCB:R_0402, F.Cu at (204.9, 101.1)
- added PB1: Tactile Button, 160gf, PCM_JLCPCB:SW-SMD_4P-L5.1-W5.1-P3.70-LS6.5-TL-2, F.Cu at (206.9, 107.1)
- added Q1: AO3401A, PCM_JLCPCB:Q_SOT-23, F.Cu at (44.0, 22.9)
- added Q2: AO3401A, PCM_JLCPCB:Q_SOT-23, F.Cu at (114.0, 73.5)
- added Q3: AO3401A, PCM_JLCPCB:Q_SOT-23, F.Cu at (43.8, 40.9)
- added Q4: AO3401A, PCM_JLCPCB:Q_SOT-23, F.Cu at (113.8, 82.9)
- added Q5: AO3401A, PCM_JLCPCB:Q_SOT-23, F.Cu at (114.1, 67.6)
- added Q6: AO3401A, PCM_JLCPCB:Q_SOT-23, F.Cu at (44.0, 32.1)
- added Q7: AO3401A, PCM_JLCPCB:Q_SOT-23, F.Cu at (114.0, 92.5)
- added R10: 5.1kΩ, PCM_JLCPCB:R_0402, F.Cu at (112.7, 23.3)
- added R11: 33Ω, PCM_JLCPCB:R_0402, F.Cu at (117.3, 24.5)
- added R12: 100kΩ, PCM_JLCPCB:R_0402, F.Cu at (83.3, 42.6)
- added R13: 33Ω, PCM_JLCPCB:R_0402, F.Cu at (120.3, 21.5)
- added R14: 10kΩ, PCM_JLCPCB:R_0402, F.Cu at (82.3, 42.6)
- added R15: 100kΩ, PCM_JLCPCB:R_0402, F.Cu at (85.3, 52.6)
- added R16: 10kΩ, PCM_JLCPCB:R_0402, F.Cu at (84.3, 52.6)
- added R17: 10MΩ, PCM_JLCPCB:R_0402, F.Cu at (24.9, 38.0)
- added R18: 10kΩ, PCM_JLCPCB:R_0402, F.Cu at (36.6, 29.8)
- added R19: 10MΩ, PCM_JLCPCB:R_0402, F.Cu at (130.5, 82.8)
- added R20: 10kΩ, PCM_JLCPCB:R_0402, F.Cu at (130.5, 87.9)
- added R21: 1MΩ, PCM_JLCPCB:R_0402, F.Cu at (28.7, 44.3)
- added R22: 1MΩ, PCM_JLCPCB:R_0402, F.Cu at (128.3, 86.8)
- added R23: 10MΩ, PCM_JLCPCB:R_0402, F.Cu at (32.7, 43.3)
- added R24: 10kΩ, PCM_JLCPCB:R_0402, F.Cu at (24.9, 28.5)
- added R25: 10MΩ, PCM_JLCPCB:R_0402, F.Cu at (121.1, 84.4)
- added R26: 10kΩ, PCM_JLCPCB:R_0402, F.Cu at (128.0, 79.6)
- added R27: 1MΩ, PCM_JLCPCB:R_0402, F.Cu at (30.7, 41.3)
- added R28: 22Ω, PCM_JLCPCB:R_0402, F.Cu at (35.5, 55.1)
- added R29: 1MΩ, PCM_JLCPCB:R_0402, F.Cu at (124.8, 84.7)
- added R30: 10kΩ, PCM_JLCPCB:R_0402, F.Cu at (200.9, 108.1)
- added R31: 10MΩ, PCM_JLCPCB:R_0402, F.Cu at (111.1, 68.6)
- added R32: 1MΩ, PCM_JLCPCB:R_0402, F.Cu at (110.8, 66.2)
- added R33: 10MΩ, PCM_JLCPCB:R_0402, F.Cu at (24.8, 23.9)
- added R34: 10kΩ, PCM_JLCPCB:R_0402, F.Cu at (30.6, 22.8)
- added R35: 10MΩ, PCM_JLCPCB:R_0402, F.Cu at (126.1, 87.9)
- added R36: 1MΩ, PCM_JLCPCB:R_0402, F.Cu at (24.8, 20.9)
- added R37: 1MΩ, PCM_JLCPCB:R_0402, F.Cu at (122.9, 87.3)
- added R38: 100kΩ, PCM_JLCPCB:R_0402, F.Cu at (80.1, 16.8)
- added R39: 10kΩ, PCM_JLCPCB:R_0402, F.Cu at (201.9, 108.1)
- added R6: 100kΩ, PCM_JLCPCB:R_0402, F.Cu at (77.3, 42.6)
- added R7: 10kΩ, PCM_JLCPCB:R_0402, F.Cu at (53.9, 88.5)
- added R8: 5.1kΩ, PCM_JLCPCB:R_0402, F.Cu at (112.7, 26.3)
- added R9: 10kΩ, PCM_JLCPCB:R_0402, F.Cu at (81.3, 42.6)
- added RST1: Tactile Button, 160gf, PCM_JLCPCB:SW-SMD_4P-L5.1-W5.1-P3.70-LS6.5-TL-2, F.Cu at (55.4, 96.6)
- added TP10: TestPoint, TestPoint:TestPoint_Pad_D1.0mm, F.Cu at (90.3, 43.0)
- added TP11: TestPoint, TestPoint:TestPoint_Pad_D1.0mm, F.Cu at (93.0, 68.1)
- added TP12: TestPoint, TestPoint:TestPoint_Pad_D1.0mm, F.Cu at (87.3, 44.0)
- added TP13: TestPoint, TestPoint:TestPoint_Pad_D1.0mm, F.Cu at (79.3, 40.6)
- added TP14: TestPoint, TestPoint:TestPoint_Pad_D1.0mm, F.Cu at (82.2, 37.0)
- added TP15: TestPoint, TestPoint:TestPoint_Pad_D1.0mm, F.Cu at (67.4, 48.0)
- added TP16: TestPoint, TestPoint:TestPoint_Pad_D1.0mm, F.Cu at (71.4, 49.0)
- added TP17: TestPoint, TestPoint:TestPoint_Pad_D1.0mm, F.Cu at (78.3, 57.3)
- added TP18: TestPoint, TestPoint:TestPoint_Pad_D1.0mm, F.Cu at (82.3, 53.6)
- added TP19: TestPoint, TestPoint:TestPoint_Pad_D1.0mm, F.Cu at (75.3, 60.3)
- added TP20: TestPoint, TestPoint:TestPoint_Pad_D1.0mm, F.Cu at (75.3, 54.3)
- added TP21: TestPoint, TestPoint:TestPoint_Pad_D1.0mm, F.Cu at (72.3, 60.3)
- added TP22: TestPoint, TestPoint:TestPoint_Pad_D1.0mm, F.Cu at (78.3, 54.3)
- added TP23: TestPoint, TestPoint:TestPoint_Pad_D1.0mm, F.Cu at (75.3, 57.3)
- added TP24: TestPoint, TestPoint:TestPoint_Pad_D1.0mm, F.Cu at (71.3, 64.3)
- added TP25: TestPoint, TestPoint:TestPoint_Pad_D1.0mm, F.Cu at (57.3, 23.2)
- added TP26: TestPoint, TestPoint:TestPoint_Pad_D1.0mm, F.Cu at (68.3, 64.3)
- added TP27: TestPoint, Connector_PinHeader_1.00mm:PinHeader_1x01_P1.00mm_Vertical, F.Cu at (211.9, 131.1)
- added TP28: TestPoint, Connector_PinHeader_1.00mm:PinHeader_1x01_P1.00mm_Vertical, F.Cu at (216.9, 100.1)
- added TP29: TestPoint, Connector_PinHeader_1.00mm:PinHeader_1x01_P1.00mm_Vertical, F.Cu at (191.9, 128.1)
- added TP30: TestPoint, Connector_PinHeader_1.00mm:PinHeader_1x01_P1.00mm_Vertical, F.Cu at (201.9, 103.1)
- added TP31: TestPoint, Connector_PinHeader_1.00mm:PinHeader_1x01_P1.00mm_Vertical, F.Cu at (214.9, 128.1)
- added TP32: TestPoint, Connector_PinHeader_1.00mm:PinHeader_1x01_P1.00mm_Vertical, F.Cu at (214.9, 103.1)
- added TP33: TestPoint, Connector_PinHeader_1.00mm:PinHeader_1x01_P1.00mm_Vertical, F.Cu at (213.9, 100.1)
- added TP34: TestPoint, Connector_PinHeader_1.00mm:PinHeader_1x01_P1.00mm_Vertical, F.Cu at (208.9, 128.1)
- added TP35: TestPoint, Connector_PinHeader_1.00mm:PinHeader_1x01_P1.00mm_Vertical, F.Cu at (211.9, 103.1)
- added TP36: TestPoint, Connector_PinHeader_1.00mm:PinHeader_1x01_P1.00mm_Vertical, F.Cu at (217.9, 103.1)
- added TP37: TestPoint, Connector_PinHeader_1.00mm:PinHeader_1x01_P1.00mm_Vertical, F.Cu at (205.9, 134.1)
- added TP38: TestPoint, Connector_PinHeader_1.00mm:PinHeader_1x01_P1.00mm_Vertical, F.Cu at (203.9, 131.1)
- added TP39: TestPoint, Connector_PinHeader_1.00mm:PinHeader_1x01_P1.00mm_Vertical, F.Cu at (211.9, 128.1)
- added TP4: TestPoint, TestPoint:TestPoint_Pad_D1.0mm, F.Cu at (102.7, 86.8)
- added TP40: TestPoint, Connector_PinHeader_1.00mm:PinHeader_1x01_P1.00mm_Vertical, F.Cu at (210.9, 100.1)
- added TP41: TestPoint, Connector_PinHeader_1.00mm:PinHeader_1x01_P1.00mm_Vertical, F.Cu at (208.9, 131.1)
- added TP42: TestPoint, Connector_PinHeader_1.00mm:PinHeader_1x01_P1.00mm_Vertical, F.Cu at (201.9, 128.1)
- added TP43: TestPoint, TestPoint:TestPoint_Pad_D1.0mm, F.Cu at (195.9, 116.1)
- added TP44: TestPoint, TestPoint:TestPoint_Pad_D1.0mm, F.Cu at (78.1, 17.8)
- added TP45: TestPoint, TestPoint:TestPoint_Pad_D1.0mm, F.Cu at (84.1, 19.8)
- added TP5: TestPoint, TestPoint:TestPoint_Pad_D1.0mm, F.Cu at (95.6, 47.1)
- added TP6: TestPoint, TestPoint:TestPoint_Pad_D1.0mm, F.Cu at (88.4, 68.0)
- added TP7: TestPoint, TestPoint:TestPoint_Pad_D1.0mm, F.Cu at (77.3, 45.6)
- added TP8: TestPoint, TestPoint:TestPoint_Pad_D1.0mm, F.Cu at (88.4, 65.0)
- added TP9: TestPoint, TestPoint:TestPoint_Pad_D1.0mm, F.Cu at (92.4, 70.0)
- added TST-R10: 0Ω, PCM_JLCPCB:R_0603, F.Cu at (32.7, 40.3)
- added TST-R11: 0Ω, PCM_JLCPCB:R_0603, F.Cu at (119.1, 84.4)
- added TST-R12: 0Ω, PCM_JLCPCB:R_0603, F.Cu at (117.9, 77.9)
- added TST-R13: 0Ω, PCM_JLCPCB:R_0603, F.Cu at (191.9, 116.1)
- added TST-R14: 0Ω, PCM_JLCPCB:R_0603, F.Cu at (39.5, 34.5)
- added TST-R15: 0Ω, PCM_JLCPCB:R_0603, F.Cu at (149.9, 128.1)
- added TST-R16: 0Ω, PCM_JLCPCB:R_0603, F.Cu at (119.1, 81.4)
- added TST-R17: 0Ω, PCM_JLCPCB:R_0603, F.Cu at (62.6, 83.3)
- added TST-R4: 0Ω, PCM_JLCPCB:R_0603, F.Cu at (102.7, 89.8)
- added TST-R5: 0Ω, PCM_JLCPCB:R_0603, F.Cu at (83.3, 45.6)
- added TST-R6: 0Ω, PCM_JLCPCB:R_0603, F.Cu at (120.3, 29.5)
- added TST-R7: 0Ω, PCM_JLCPCB:R_0603, F.Cu at (31.9, 36.0)
- added TST-R8: 0Ω, PCM_JLCPCB:R_0603, F.Cu at (131.1, 79.3)
- added TST-R9: 0Ω, PCM_JLCPCB:R_0603, F.Cu at (59.2, 26.1)
- added U1: MT9221CT-06BR5, JLCPCB:Current-sensor_MT9221CT-06BR5_C879632, F.Cu at (112.1, 100.5)
- added U3: USBLC6-2SC6, Package_TO_SOT_SMD:SOT-23-6, F.Cu at (108.0, 29.4)
- added U4: ESP32-S3, PCM_JLCPCB:QFN-56-1EP_7x7mm_P0.4mm_EP4x4mm_ThermalVias, F.Cu at (87.3, 58.2)
- added U5: AXP2101, Package_DFN_QFN:QFN-40-1EP_5x5mm_P0.4mm_EP3.6x3.6mm_ThermalVias, F.Cu at (207.3, 115.1)
- added U6: DS18B20U(UMW), JLCPCB:DS18B20_C695836, F.Cu at (67.6, 82.1)
- added U7: W25Q128JVSIQ, PCM_JLCPCB:SOIC-8_L5.3-W5.3-P1.27-LS8.0-BL, F.Cu at (90.5, 21.1)
- added Y1: 40MHz, 15pF, JLCPCB:OSC-SMD_4P-L3.2-W2.5-BL_SIT8008BI, F.Cu at (28.5, 58.1)
- added Y2: 32.768KHz, Crystal:Crystal_SMD_3215-2Pin_3.2x1.5mm, F.Cu at (37.8, 58.1)
- moved C59 59.7 mm to (95.2, 181.6)
- moved C62 59.7 mm to (123.9, 174.8)
- moved J17 59.7 mm to (108.4, 152.9)
- moved J18 59.7 mm to (108.4, 170.7)
- moved JP7 59.7 mm to (127.6, 178.7)
- moved PB2 59.7 mm to (123.7, 184.5)
- moved PB3 59.7 mm to (117.6, 190.6)
- moved PB4 59.7 mm to (117.6, 178.4)
- moved TST-R23 59.7 mm to (123.9, 177.4)
- moved TST-R24 59.7 mm to (123.9, 176.1)
- moved U11 59.7 mm to (127.7, 175.5)
- moved C55 59.7 mm to (38.1, 188.2)
- moved C61 59.7 mm to (35.8, 177.1)
- moved TP49 59.7 mm to (40.4, 192.4)
- moved TST-R19 59.7 mm to (36.6, 188.1)
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- renumbered C66 to C53, C67 to C56, C43 to C57, C44 to C58, C45 to C59, C47 to C60, C69 to C61, C70 to C62, J10 to J16, J2 to J17, J1 to J18, JP3 to JP1, JP1 to JP2, JP4 to JP3, JP5 to JP4, JP6 to JP5, JP7 to JP6, JP8 to JP7, PB4 to PB2, PB5 to PB3, PB1 to PB4, PB2 to PB5, R43 to R42, R38 to R43, R39 to R44, TP1 to TP46, TP66 to TP47, TP63 to TP48, TP67 to TP49, TP64 to TP50, TP85 to TP51, TP56 to TP52, TP47 to TP53, TP57 to TP54, TP49 to TP55, TST-R16 to TST-R18, TST-R18 to TST-R19, TST-R14 to TST-R20, TST-R20 to TST-R21, TST-R26 to TST-R22, TST-R21 to TST-R23, TST-R27 to TST-R24, U16 to U10, U17 to U11, U15 to U8, U11 to U9
Other:
- board size 97.5 x 45.7 mm -> 244.5 x 128.3 mm

Commit message: Reverted Smaller
Parts:
- removed ANT1: KH-3216-H0209, JLCPCB:ANT-SMD_L3.2-W1.6-KH-3216F245C04
- removed BOOT1, RST1: Tactile Button, 160gf, PCM_JLCPCB:SW-SMD_4P-L5.1-W5.1-P3.70-LS6.5-TL-2
- removed BT1: BH-18650-B1BA002, JLCPCB:BATTERY-SMD_18650-1S-L77.1-W20.7-1
- removed C1, C12, C13, C14, C15, C16, C17, C18, C37, C49, C8, C9: 100nF, PCM_JLCPCB:C_0603
- removed C10, C26: 10uF, PCM_JLCPCB:C_0402
- removed C11, C38: 1uF, PCM_JLCPCB:C_0603
- removed C19, C20: 3.3pF, PCM_JLCPCB:C_0402
- removed C2: 1nF, PCM_JLCPCB:C_0402
- removed C21, C23: 10pF, PCM_JLCPCB:C_0402
- removed C22, C28, C30, C40, C46, C48: 1uF, PCM_JLCPCB:C_0402
- removed C24, C25: 20pF, PCM_JLCPCB:C_0402
- removed C27, C29, C31, C33, C52: 22uF, PCM_JLCPCB:C_0603
- removed C32, C34, C35, C36, C41, C42, C50, C51: 2.2uF, PCM_JLCPCB:C_0402
- removed C39: 4.7uF, PCM_JLCPCB:C_0402
- removed the C43 at (216.9, 114.1)
- removed the C44 at (211.9, 109.1)
- removed the C45 at (215.9, 117.1)
- removed the C47 at (214.9, 114.1)
- removed D1: 1N4148W, PCM_JLCPCB:D_SOD-123
- removed D2, D5, D6, D8: IR, JLCPCB:IR-LED_C131280
- removed D3: White, PCM_JLCPCB:D_0603
- removed D4: WS2812B, PCM_JLCPCB:LED-SMD_4P-L1.6-W1.5_XL-1615RGBC-WS2812B
- removed D7: Yellow, PCM_JLCPCB:D_0805
- removed D9: Green, PCM_JLCPCB:D_0805
- removed the J1 at (128.7, 26.0)
- removed the J10 at (135.2, 78.3)
- removed J11, J14, J7, J8: Conn_01x03, Connector_PinHeader_2.54mm:PinHeader_1x03_P2.54mm_Vertical
- removed J12, J13, J15, J3, J4, J5, J6, J9: Conn_01x02, Connector_PinHeader_1.00mm:PinHeader_1x02_P1.00mm_Vertical
- removed the J2 at (35.6, 26.8)
- removed L3, L4: 2nH, Inductor_SMD:L_0603_1608Metric_Pad1.05x0.95mm_HandSolder
- removed L5, L6, L7, L8, L9: 1uH,3.3A, Inductor_SMD:L_1008_2520Metric
- removed NTC1: NTC, PCM_JLCPCB:R_0402
- removed the PB1 at (206.9, 107.1)
- removed Q1, Q2, Q3, Q4, Q5, Q6, Q7: AO3401A, PCM_JLCPCB:Q_SOT-23
- removed R10, R8: 5.1kΩ, PCM_JLCPCB:R_0402
- removed R11, R13: 33Ω, PCM_JLCPCB:R_0402
- removed R12, R15, R6: 100kΩ, PCM_JLCPCB:R_0402
- removed R14, R16, R18, R20, R24, R26, R30, R34, R7, R9: 10kΩ, PCM_JLCPCB:R_0402
- removed R17, R19, R23, R25, R31, R33, R35: 10MΩ, PCM_JLCPCB:R_0402
- removed R21, R22, R27, R29, R32, R36, R37: 1MΩ, PCM_JLCPCB:R_0402
- removed R28: 22Ω, PCM_JLCPCB:R_0402
- removed the R38 at (80.1, 16.8)
- removed the R39 at (201.9, 108.1)
- removed TP10, TP11, TP12, TP13, TP14, TP15, TP16, TP17, TP18, TP19, TP20, TP21, TP22, TP23, TP24, TP25, TP26, TP4, TP43, TP44, TP45, TP5, TP6, TP7, TP8, TP9: TestPoint, TestPoint:TestPoint_Pad_D1.0mm
- removed TP27, TP28, TP29, TP30, TP31, TP32, TP33, TP34, TP35, TP36, TP37, TP38, TP39, TP40, TP41, TP42: TestPoint, Connector_PinHeader_1.00mm:PinHeader_1x01_P1.00mm_Vertical
- removed TST-R10, TST-R11, TST-R12, TST-R13, TST-R15, TST-R17, TST-R4, TST-R5, TST-R6, TST-R7, TST-R8, TST-R9: 0Ω, PCM_JLCPCB:R_0603
- removed the TST-R14 at (39.5, 34.5)
- removed the TST-R16 at (119.1, 81.4)
- removed U1: MT9221CT-06BR5, JLCPCB:Current-sensor_MT9221CT-06BR5_C879632
- removed U3: USBLC6-2SC6, Package_TO_SOT_SMD:SOT-23-6
- removed U4: ESP32-S3, PCM_JLCPCB:QFN-56-1EP_7x7mm_P0.4mm_EP4x4mm_ThermalVias
- removed U5: AXP2101, Package_DFN_QFN:QFN-40-1EP_5x5mm_P0.4mm_EP3.6x3.6mm_ThermalVias
- removed U6: DS18B20U(UMW), JLCPCB:DS18B20_C695836
- removed U7: W25Q128JVSIQ, PCM_JLCPCB:SOIC-8_L5.3-W5.3-P1.27-LS8.0-BL
- removed Y1: 40MHz, 15pF, JLCPCB:OSC-SMD_4P-L3.2-W2.5-BL_SIT8008BI
- removed Y2: 32.768KHz, Crystal:Crystal_SMD_3215-2Pin_3.2x1.5mm
- moved C45 59.7 mm to (144.1, 147.3)
- moved C70 59.7 mm to (172.8, 140.5)
- moved J1 59.7 mm to (157.3, 136.4)
- moved J2 59.7 mm to (157.3, 118.6)
- moved JP8 59.7 mm to (176.6, 144.3)
- moved PB1 59.7 mm to (166.5, 144.1)
- moved PB4 59.7 mm to (172.6, 150.2)
- moved PB5 59.7 mm to (166.5, 156.3)
- moved TST-R21 59.7 mm to (172.8, 143.1)
- moved TST-R27 59.7 mm to (172.8, 141.8)
- moved U17 59.7 mm to (176.6, 141.2)
- moved C55 59.7 mm to (87.0, 153.9)
- moved C69 59.7 mm to (84.7, 142.8)
- moved TP67 59.7 mm to (89.3, 158.1)
- moved TST-R18 59.7 mm to (85.6, 153.8)
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- renumbered C57 to C43, C58 to C44, C59 to C45, C60 to C47, C53 to C66, C56 to C67, C61 to C69, C62 to C70, J18 to J1, J16 to J10, J17 to J2, JP2 to JP1, JP1 to JP3, JP3 to JP4, JP4 to JP5, JP5 to JP6, JP6 to JP7, JP7 to JP8, PB4 to PB1, PB5 to PB2, PB2 to PB4, PB3 to PB5, R43 to R38, R44 to R39, R42 to R43, TP46 to TP1, TP53 to TP47, TP55 to TP49, TP52 to TP56, TP54 to TP57, TP48 to TP63, TP50 to TP64, TP47 to TP66, TP49 to TP67, TP51 to TP85, TST-R20 to TST-R14, TST-R18 to TST-R16, TST-R19 to TST-R18, TST-R21 to TST-R20, TST-R23 to TST-R21, TST-R22 to TST-R26, TST-R24 to TST-R27, U9 to U11, U8 to U15, U10 to U16, U11 to U17
Other:
- board size 244.5 x 128.3 mm -> 97.5 x 45.7 mm
