File: ESP32S3_Audio_Cam_POE_Smaller.kicad_sch (KiCad schematic)
At the start: 50 parts, among them CN1 PJ-316C-6A, J1 Conn_01x20_Pin, J10 Conn_01x02, J2 Conn_01x20_Pin, U11 TM1637, U15 MAX98357AETE+T, U16 ICS-43434, U17 ICS-43434

Commit message: Draft smaller board.
Parts:
- added JP1: SolderJumper_3_Bridged12, Jumper:SolderJumper-3_P1.3mm_Bridged12_Pad1.0x1.5mm, symbol Jumper:SolderJumper_3_Bridged12
- added TP1: TestPoint, Connector_PinHeader_1.00mm:PinHeader_1x01_P1.00mm_Vertical, symbol Connector:TestPoint
Connections:
- net COM: now also JP1.3 (B)
- net SPK.BCLK: now also J1.16 (Pin_16); no longer J1.15 (Pin_15)
- net SPK.DIN: now also J1.15 (Pin_15); no longer J1.16 (Pin_16)
- net SPK.LRCLK: now also JP1.2 (C), TP1.1
- net V.SPK: now reaches C54.1, C55.1, TST-R18.1, U15.7 (VDD), U15.8 (VDD)
- net V.SPK: now also JP1.1 (A)

Commit message: Draft
Parts:
- added ANT1: KH-3216-H0209, JLCPCB:ANT-SMD_L3.2-W1.6-KH-3216F245C04, symbol JLCPCB-Extended:KH-3216-H0209_C2925417
- added BOOT1, PB1, RST1: Tactile Button, 160gf, PCM_JLCPCB:SW-SMD_4P-L5.1-W5.1-P3.70-LS6.5-TL-2, symbol PCM_JLCPCB-Connectors_Buttons:Tactile Button, 160gf
- added BT1: BH-18650-B1BA002, JLCPCB:BATTERY-SMD_18650-1S-L77.1-W20.7-1, symbol JLCPCB-Extended:BH-18650-B1BA002_18650_C2988620
- added C1, C12, C13, C14, C15, C16, C17, C18, C37, C49, C8, C9: 100nF, PCM_JLCPCB:C_0603, symbol PCM_JLCPCB-Capacitors:0603,100nF
- added C10: 10uF, PCM_JLCPCB:C_0402, symbol PCM_JLCPCB-Capacitors:0402,10uF
- added C11, C38: 1uF, PCM_JLCPCB:C_0603, symbol PCM_JLCPCB-Capacitors:0603,1uF
- added C19, C20: 3.3pF, PCM_JLCPCB:C_0402, symbol PCM_JLCPCB-Capacitors:0402,3.3pF
- added C2: 1nF, PCM_JLCPCB:C_0402, symbol JLCPCB-Capacitors:0402,1nF
- added C21, C23: 10pF, PCM_JLCPCB:C_0402, symbol PCM_JLCPCB-Capacitors:0402,10pF
- added C22, C28, C30, C40, C45, C46, C48: 1uF, PCM_JLCPCB:C_0402, symbol JLCPCB-Capacitors:0402,1uF
- added C24, C25: 20pF, PCM_JLCPCB:C_0402, symbol PCM_JLCPCB-Capacitors:0402,20pF
- added C26: 10uF, PCM_JLCPCB:C_0402, symbol JLCPCB-Capacitors:0402,10uF
- added C27, C29, C31, C33, C44, C52: 22uF, PCM_JLCPCB:C_0603, symbol JLCPCB-Capacitors:0603,22uF
- added C32, C34, C35, C36, C41, C42, C43, C47, C50, C51: 2.2uF, PCM_JLCPCB:C_0402, symbol JLCPCB-Capacitors:0402,2.2uF
- added C39: 4.7uF, PCM_JLCPCB:C_0402, symbol JLCPCB-Capacitors:0402,4.7uF
- added D1: 1N4148W, PCM_JLCPCB:D_SOD-123, symbol PCM_JLCPCB-Diodes:Switching,1N4148W
- added D2, D5, D6, D8: IR, JLCPCB:IR-LED_C131280, symbol JLCPCB-Diodes:LED IR IR26-21c_C131280
- added D3: White, PCM_JLCPCB:D_0603, symbol JLCPCB-Diodes:LED,0603,White
- added D4: WS2812B, PCM_JLCPCB:LED-SMD_4P-L1.6-W1.5_XL-1615RGBC-WS2812B, symbol JLCPCB-Extended:LED, WS2812B, 1615
- added D7: Yellow, PCM_JLCPCB:D_0805, symbol JLCPCB-Diodes:LED,0805,Yellow
- added D9: Green, PCM_JLCPCB:D_0805, symbol PCM_JLCPCB-Diodes:LED,0805,Green
- added J1: Connector, USB-TYPE-C-16P, PCM_JLCPCB:TYPE-C-SMD_HX-TYPE-C-16PIN, symbol PCM_JLCPCB-Extended:Connector, USB-TYPE-C-16P
- added J10, J12, J13, J15, J2, J3, J4, J5, J6, J9: Conn_01x02, Connector_PinHeader_1.00mm:PinHeader_1x02_P1.00mm_Vertical, symbol Connector_Generic:Conn_01x02
- added J11, J14, J7, J8: Conn_01x03, Connector_PinHeader_2.54mm:PinHeader_1x03_P2.54mm_Vertical, symbol Connector_Generic:Conn_01x03
- added L3, L4: 2nH, Inductor_SMD:L_0603_1608Metric_Pad1.05x0.95mm_HandSolder, symbol Device:L
- added L5, L6, L7, L8, L9: 1uH,3.3A, Inductor_SMD:L_1008_2520Metric, symbol JLCPCB-Inductors:1uH,50mA
- added NTC1: NTC, PCM_JLCPCB:R_0402, symbol JLCPCB-Resistors:0402,10kΩ
- added Q1, Q2, Q3, Q4, Q5, Q6, Q7: AO3401A, PCM_JLCPCB:Q_SOT-23, symbol PCM_JLCPCB-Transistors:PMOS,AO3401A
- added R10, R8: 5.1kΩ, PCM_JLCPCB:R_0402, symbol PCM_JLCPCB-Resistors:0402,5.1kΩ
- added R11, R13: 33Ω, PCM_JLCPCB:R_0402, symbol PCM_JLCPCB-Resistors:0402,33Ω
- added R12, R15, R38, R6: 100kΩ, PCM_JLCPCB:R_0402, symbol PCM_JLCPCB-Resistors:0402,100kΩ
- added R14, R16, R18, R20, R24, R26, R30, R34, R39, R7, R9: 10kΩ, PCM_JLCPCB:R_0402, symbol PCM_JLCPCB-Resistors:0402,10kΩ
- added R17, R19, R23, R25, R31, R33, R35: 10MΩ, PCM_JLCPCB:R_0402, symbol PCM_JLCPCB-Resistors:0402,10MΩ
- added R21, R22, R27, R29, R32, R36, R37: 1MΩ, PCM_JLCPCB:R_0402, symbol PCM_JLCPCB-Resistors:0402,1MΩ
- added R28: 22Ω, PCM_JLCPCB:R_0402, symbol PCM_JLCPCB-Resistors:0402,22Ω
- added TP10, TP11, TP12, TP13, TP14, TP15, TP16, TP17, TP18, TP19, TP20, TP21, TP22, TP23, TP24, TP25, TP26, TP4, TP43, TP44, TP45, TP5, TP6, TP7, TP8, TP9: TestPoint, TestPoint:TestPoint_Pad_D1.0mm, symbol Connector:TestPoint
- added TP27, TP28, TP29, TP30, TP31, TP32, TP33, TP34, TP35, TP36, TP37, TP38, TP39, TP40, TP41, TP42: TestPoint, Connector_PinHeader_1.00mm:PinHeader_1x01_P1.00mm_Vertical, symbol Connector:TestPoint
- added TST-R10, TST-R11, TST-R12, TST-R13, TST-R14, TST-R15, TST-R16, TST-R17, TST-R4, TST-R5, TST-R6, TST-R7, TST-R8, TST-R9: 0Ω, PCM_JLCPCB:R_0603, symbol PCM_JLCPCB-Resistors:0603,0Ω
- added U1: MT9221CT-06BR5, JLCPCB:Current-sensor_MT9221CT-06BR5_C879632, symbol JLCPCB-Extended:Current-sensor_MT9221CT-06BR5_C879632
- added U3: USBLC6-2SC6, Package_TO_SOT_SMD:SOT-23-6, symbol Power_Protection:USBLC6-2SC6
- added U4: ESP32-S3, PCM_JLCPCB:QFN-56-1EP_7x7mm_P0.4mm_EP4x4mm_ThermalVias, symbol PCM_JLCPCB-Extended:MCU, ESP32-S3
- added U5: AXP2101, Package_DFN_QFN:QFN-40-1EP_5x5mm_P0.4mm_EP3.6x3.6mm_ThermalVias, symbol JLCPCB-Extended:AXP2101_C3036461
- added U6: DS18B20U(UMW), JLCPCB:DS18B20_C695836, symbol JLCPCB-ICs:DS18B20_C695836
- added U7: W25Q128JVSIQ, PCM_JLCPCB:SOIC-8_L5.3-W5.3-P1.27-LS8.0-BL, symbol PCM_JLCPCB-Memory:16MByte, SPI
- added Y1: 40MHz, 15pF, JLCPCB:OSC-SMD_4P-L3.2-W2.5-BL_SIT8008BI, symbol JLCPCB-Extended:Crystal, 40MHz, 15pF
- added Y2: 32.768KHz, Crystal:Crystal_SMD_3215-2Pin_3.2x1.5mm, symbol Device:Crystal
- renumbered C66 to C53, C67 to C56, C43 to C57, C44 to C58, C45 to C59, C47 to C60, C69 to C61, C70 to C62, J10 to J16, J2 to J17, J1 to J18, JP3 to JP1, JP1 to JP2, JP4 to JP3, JP5 to JP4, JP6 to JP5, JP7 to JP6, JP8 to JP7, PB4 to PB2, PB5 to PB3, PB1 to PB4, PB2 to PB5, R43 to R42, R38 to R43, R39 to R44, TP1 to TP46, TP66 to TP47, TP63 to TP48, TP67 to TP49, TP64 to TP50, TP85 to TP51, TP56 to TP52, TP47 to TP53, TP57 to TP54, TP49 to TP55, TST-R16 to TST-R18, TST-R18 to TST-R19, TST-R14 to TST-R20, TST-R20 to TST-R21, TST-R26 to TST-R22, TST-R21 to TST-R23, TST-R27 to TST-R24, U16 to U10, U17 to U11, U15 to U8, U11 to U9
Connections:
- net +3V3: now also C10.1, C9.2, L3.2, R6.2, R7.2, TST-R13.2, TST-R17.1, TST-R5.2, TST-R9.2
- net COM: now also BOOT1.3 (C), BT1.1, C1.2, C10.2, C11.1, C12.2, C13.2, C14.2, C15.2, C16.1, C17.1, C18.1, C19.2, C2.2, C20.2, C21.2, C22.1, C23.2, C24.2, C25.2, C26.2, C27.1, C28.1, C29.1, C30.1, C31.1, C32.1, C33.1, C34.1, C35.1, C36.1, C37.1, C38.2, C39.1, C40.1, C41.1, C42.1, C43.1, C44.1, C45.1, C46.1, C47.1, C48.1, C49.1, C50.1, C51.1, C52.1, C8.1, C9.1, D2.1 (C), D3.1, D4.3 (GND), D5.1 (C), D6.1 (C), D8.1 (C), J1.A12B1 (GND), J1.B12A1 (GND), J1.S1 (SHIELD), J10.2 (Pin_2), J11.3 (Pin_3), J12.2 (Pin_2), J13.2 (Pin_2), J14.3 (Pin_3), J15.2 (Pin_2), J2.2 (Pin_2), J3.2 (Pin_2), J5.2 (Pin_2), J6.2 (Pin_2), J7.3 (Pin_3), J8.3 (Pin_3), J9.2 (Pin_2), NTC1.1, PB1.3 (C), R10.2, R14.2, R16.2, R8.2, R9.2, RST1.3 (C), U1.5 (GND), U3.2 (GND), U4.57 (GND), U5.3 (GND), U5.41 (EP), U6.4 (GND), U7.4 (GND), Y1.2 (GND), Y1.4 (GND)
- net Vdrive: now also TST-R10.2, TST-R11.2, TST-R12.2, TST-R14.2, TST-R15.2, TST-R16.1, TST-R7.2, TST-R8.2, U1.1 (IP+), U1.2 (IP+)
- new net: D6.2 (A), R26.2
- new net: Q5.2 (S), R31.1, TST-R12.1
- new net: Q5.1 (G), R31.2, R32.1
- new net: Q3.2 (S), R23.1, TST-R10.1
- new net: Q3.1 (G), R23.2, R27.1
- new net: J9.1 (Pin_1), Q6.3 (D), R34.1
- new net: D1.2, J1.A9B4 (VBUS), J1.B9A4 (VBUS)
- new net: Q7.1 (G), R35.2, R37.1
- new net: Q2.2 (S), R19.1, TST-R8.1
- new net: Q2.1 (G), R19.2, R22.1
- new net: D7.2, R30.1
- new net: Q1.1 (G), R17.2, R21.1
- new net: Q6.1 (G), R33.2, R36.1
- new net: C26.1, TST-R15.1, U5.37 (VBUS)
- new net: D3.2, R20.2
- new net: D7.1, U5.1 (CHGLED)
- new net: L9.2, U5.21 (FB1)
- new net: L8.2, U5.25 (LX2)
- new net: J15.1 (Pin_1), U5.27 (VBACKUP)
- new net: C40.2, U5.28 (VRTC)
- new net: D9.1, U5.29 (PWROK)
- new net: PB1.1 (A), U5.30 (PWRON)
- new net: J13.1 (Pin_1), NTC1.2, U5.31 (TS)
- new net: BT1.2, C32.2, J12.1 (Pin_1), U5.33 (BAT)
- new net: L6.2, U5.35 (SW)
- new net: TP43.1, U5.38 (IRQ)
- new net: L5.2, U5.5 (LX3)
- new net: L7.2, U5.9 (FB4)
- new net: J3.1 (Pin_1), Q2.3 (D), R20.1
- new net: C11.2, C12.1, C13.1, C14.1, C15.1, TST-R5.1, U4.2 (VDD3P3), U4.20 (VDD3P3_RTC), U4.3 (VDD3P3), U4.55 (VDDA), U4.56 (VDDA)
- new net: D9.2, R39.1
- new net: Q4.1 (G), R25.2, R29.1
- new net: D8.2 (A), R34.2
- new net: Q7.2 (S), R35.1, TST-R16.2
- new net: J10.1 (Pin_1), Q7.3 (D)
- new net: L3.1, TP4.1, TST-R4.2
- new net: Q6.2 (S), R33.1, TST-R14.1
- new net: J2.1 (Pin_1), Q1.3 (D), R18.1
- new net: D2.2 (A), R18.2
- new net: C18.2, D4.2 (VDD), TST-R9.1
- new net: J5.1 (Pin_1), Q3.3 (D), R24.1
- new net: D5.2 (A), R24.2
- new net: C23.1, R28.1, Y1.1 (OSC)
- new net: TST-R6.2, U3.5 (VBUS)
- new net: C49.2, TST-R17.2, U6.8 (VDD)
- new net: Q1.2 (S), R17.1, TST-R7.1
- new net: Q4.2 (S), R25.1, TST-R11.1
- new net: J6.1 (Pin_1), Q4.3 (D), R26.1
- new net +3V3_RF2: C8.2, TST-R4.1, U4.46 (VDD3P3_CPU)
- new net 2CHIP_BOOT: BOOT1.1 (A), C16.2, U4.5 (GPIO0)
- new net 2CHIP_PU: C17.2, R7.1, RST1.1 (A), U4.4 (CHIP_PU)
- new net 2FLASH_QSPI_CLK: U4.33 (SPICLK), U7.6 (CLK)
- new net 2FLASH_QSPI_DI: U4.35 (SPID), U7.5 (DI)
- new net 2FLASH_QSPI_DO: U4.34 (SPIQ), U7.2 (DO)
- new net 2FLASH_QSPI_nCS: R38.1, TP44.1, U4.32 (SPICS0), U7.1 (CS#)
- new net 2FLASH_QSPI_nH: U4.30 (SPIHD), U7.7 (IO3)
- new net 2FLASH_QSPI_nWP: U4.31 (SPIWP), U7.3 (IO2)
- new net 2GPIO1: TP6.1, U4.6 (GPIO1)
- new net 2GPIO3: TP8.1, U4.8 (GPIO3)
- new net 2GPIO39: TP20.1, U4.44 (MTCK)
- new net 2GPIO40: TP21.1, U4.45 (MTDO)
- new net 2GPIO41: TP22.1, U4.47 (MTDI)
- new net 2GPIO42: TP23.1, U4.48 (MTMS)
- new net 2GPIO45: TP24.1, U4.51 (GPIO45)
- new net 2GPIO46: TP26.1, U4.52 (GPIO46)
- new net 2GPIO47: TP12.1, U4.37 (SPICLK_P)
- new net 2GPIO48: TP10.1, U4.36 (SPICLK_N)
- new net 2GPIO7: TP9.1, U4.12 (GPIO7)
- new net 2GPIO8: TP11.1, U4.13 (GPIO8)
- new net 2OSC32_IN: C24.1, U4.21 (XTAL_32K_P), Y2.1
- new net 2OSC32_OUT: C25.1, U4.22 (XTAL_32K_N), Y2.2
- new net 2OSC_IN: R28.2, U4.54 (XTAL_P)
- new net 2OSC_OUT: C21.1, U4.53 (XTAL_N), Y1.3 (OSC)
- new net 2U0RXD: J4.2 (Pin_2), U4.50 (U0RXD)
- new net 2U0TXD: J4.1 (Pin_1), U4.49 (U0TXD)
- new net 2USB_CC1: J1.A5 (CC1), R8.1
- new net 2USB_CC2: J1.B5 (CC2), R10.1
- new net 2USB_D+: R13.2, U3.3 (I/O2), U3.4 (I/O2), U4.26 (GPIO20/USB_D+)
- new net 2USB_D-: R11.2, U3.1 (I/O1), U3.6 (I/O1), U4.25 (GPIO19/USB_D-)
- new net 2USB_PRT_D+: J1.A6 (D+), J1.B6 (D+), R13.1
- new net 2USB_PRT_D-: J1.A7 (D-), J1.B7 (D-), R11.1
- new net 2VDD_SPI: C37.2, C38.1, R38.2, TP45.1, U4.29 (VDD_SPI), U7.8 (VCC)
- new net 3v3.Sense: R6.1, R9.1, TP7.1, U4.7 (GPIO2)
- new net ISEN.FLT: C2.1, U1.6 (FILTER)
- new net ISEN.VO: U1.7 (VOUT), U4.23 (GPIO17)
- new net LED.IR: R29.2, U4.10 (GPIO5)
- new net LED.OTH: R37.2, U4.11 (GPIO6)
- new net LED.RGB: D4.4 (DIN), TP25.1, U4.27 (GPIO21)
- new net LED.WH: R22.2, U4.9 (GPIO4)
- new net MISC.OUT1: R36.2, TP14.1, U4.39 (GPIO34)
- new net MISC.OUT2: R27.2, TP15.1, U4.40 (GPIO35)
- new net MISC.OUT3: R21.2, TP16.1, U4.41 (GPIO36)
- new net PMU.SCK: TP17.1, U4.42 (GPIO37), U5.39 (SCK)
- new net PMU.SDA: TP19.1, U4.43 (GPIO38), U5.40 (SDA)
- new net PMU.Va1: C47.2, TP28.1, U5.18 (ALDO1)
- new net PMU.Va2: C50.2, TP32.1, U5.19 (ALDO2)
- new net PMU.Va3: C43.2, TP36.1, U5.16 (ALDO3)
- new net PMU.Va4: C42.2, TP40.1, U5.15 (ALDO4)
- new net PMU.Vb1: C36.2, TP27.1, U5.12 (BLDO1)
- new net PMU.Vb2: C41.2, TP31.1, U5.14 (BLDO2)
- new net PMU.Vcpu: C34.2, TP34.1, U5.10 (CPULDOS)
- new net PMU.Vd1: C51.2, TP35.1, U5.20 (DLDO1/DC1SW)
- new net PMU.Vd2: C35.2, TP39.1, U5.11 (DLDO2/DC4SW)
- new net PMU.Vo1: C52.2, L9.1, R12.2, TP29.1, TST-R13.1, U5.22 (LX1)
- new net PMU.Vo1.Sense: R12.1, R14.1, TP13.1, U4.38 (GPIO33)
- new net PMU.Vo2: C44.2, L8.1, TP33.1, U5.26 (FB2)
- new net PMU.Vo3: C27.2, L5.1, TP37.1, U5.4 (FB3)
- new net PMU.Vo4: C33.2, L7.1, TP41.1, U5.8 (LX4)
- new net PMU.Vref: C22.2, TP38.1, TP5.1, U4.28 (SPICS1), U5.2 (VREF)
- new net PMU.Vsys: C28.2, C30.2, C39.2, C45.2, C46.2, C48.2, R30.2, R39.2, TP30.1, U5.13 (BLDOIN), U5.17 (ALDOIN), U5.23 (VIN1), U5.24 (VIN2), U5.34 (VSYS), U5.36 (VMID), U5.6 (VIN3), U5.7 (VIN4)
- new net RC.OTHR: J14.1 (Pin_1), U4.18 (GPIO13)
- new net RC.PAN: J7.1 (Pin_1), U4.15 (GPIO10)
- new net RC.PWR: R32.2, U4.14 (GPIO9)
- new net RC.ROT: J11.1 (Pin_1), U4.17 (GPIO12)
- new net RC.TILT: J8.1 (Pin_1), U4.16 (GPIO11)
- new net RC.VDD: J11.2 (Pin_2), J14.2 (Pin_2), J7.2 (Pin_2), J8.2 (Pin_2), Q5.3 (D)
- new net RF2: C19.1, L4.1, U4.1 (LNA_IN)
- new net RF2-ANT: ANT1.1 (ANT), C20.1, L4.2
- new net TEMP.DQ: U4.24 (GPIO18), U6.1 (DQ)
- new net VBUS: C1.1, D1.1, R15.2, TST-R6.1, U1.3 (IP-), U1.4 (IP-), U1.8 (VCC)
- new net VBus.Sense: R15.1, R16.1, TP18.1, U4.19 (GPIO14)
- new net VDCDC5: C29.2, C31.2, L6.1, TP42.1, U5.32 (GPIO1/FB5/RTC/LDO2)
- no-connect marks 8 -> 23
Other:
- note added: "(CL(Load) - Cs(Stray)) * 2 = Capacitance (10p - +/-4p) * 2 = 10p"
- note added: "2GPIO10"
- note added: "2GPIO11"
- note added: "2GPIO12"
- note added: "2GPIO13"
- note added: "2GPIO14"
- note added: "2GPIO15"
- note added: "2GPIO16"
- note added: "2GPIO17"
- note added: "2GPIO18"
- note added: "2GPIO19"
- note added: "2GPIO2"
- note added: "2GPIO20"
- note added: "2GPIO21"
- note added: "2GPIO26"
- note added: "2GPIO27"
- note added: "2GPIO28"
- note added: "2GPIO29"
- note added: "2GPIO30"
- note added: "2GPIO31"
- note added: "2GPIO32"
- note added: "2GPIO33"
- note added: "2GPIO34"
- note added: "2GPIO35"
- note added: "2GPIO36"
- note added: "2GPIO37"
- note added: "2GPIO38"
- note added: "2GPIO4"
- note added: "2GPIO43"
- note added: "2GPIO44"
- note added: "2GPIO5"
- note added: "2GPIO6"
- note added: "2GPIO9"
- note added: "2USB_C"
- note added: "BATTERY PMU / GUAGE"
- note added: "Boot Button"
- note added: "Crystals"
- note added: "Current Sense"
- note added: "FC = 1/(2*PI*Rfint*Cfilter) 88Hz = 1/(2*PI*1.8kohm*1nF)"
- note added: "HSE / LSE"
- note added: "LIGHTS"
- note added: "MISC OUTPUTS"
- note added: "Mode: QuadSPI"
- note added: "NOR FLASH"
- note added: "NP = Normal P = Directly in Flash"
- note added: "NTC wants to be TH11-3H103F while C3018545 is probably a close enough equiv."
- note added: "OTHER"
- note added: "PAN"
- note added: "PCB TEMPERATURE"
- note added: "PI Filter Antenna"
- note added: "Pull-Up"
- note added: "RC SERVO'S"
- note added: "RF Voltage Filter"
- note added: "RGB Status LED"
- note added: "ROTATE"
- note added: "RST Button"
- note added: "TILT"
- note added: "Z=(35+j10)R"
- note added: "Z=50R"

Commit message: Reverted Smaller
Parts:
- removed ANT1: KH-3216-H0209, JLCPCB:ANT-SMD_L3.2-W1.6-KH-3216F245C04, symbol JLCPCB-Extended:KH-3216-H0209_C2925417
- removed BOOT1, PB1, RST1: Tactile Button, 160gf, PCM_JLCPCB:SW-SMD_4P-L5.1-W5.1-P3.70-LS6.5-TL-2, symbol PCM_JLCPCB-Connectors_Buttons:Tactile Button, 160gf
- removed BT1: BH-18650-B1BA002, JLCPCB:BATTERY-SMD_18650-1S-L77.1-W20.7-1, symbol JLCPCB-Extended:BH-18650-B1BA002_18650_C2988620
- removed C1, C12, C13, C14, C15, C16, C17, C18, C37, C49, C8, C9: 100nF, PCM_JLCPCB:C_0603, symbol PCM_JLCPCB-Capacitors:0603,100nF
- removed C10: 10uF, PCM_JLCPCB:C_0402, symbol PCM_JLCPCB-Capacitors:0402,10uF
- removed C11, C38: 1uF, PCM_JLCPCB:C_0603, symbol PCM_JLCPCB-Capacitors:0603,1uF
- removed C19, C20: 3.3pF, PCM_JLCPCB:C_0402, symbol PCM_JLCPCB-Capacitors:0402,3.3pF
- removed C2: 1nF, PCM_JLCPCB:C_0402, symbol JLCPCB-Capacitors:0402,1nF
- removed C21, C23: 10pF, PCM_JLCPCB:C_0402, symbol PCM_JLCPCB-Capacitors:0402,10pF
- removed C22, C28, C30, C40, C45, C46, C48: 1uF, PCM_JLCPCB:C_0402, symbol JLCPCB-Capacitors:0402,1uF
- removed C24, C25: 20pF, PCM_JLCPCB:C_0402, symbol PCM_JLCPCB-Capacitors:0402,20pF
- removed C26: 10uF, PCM_JLCPCB:C_0402, symbol JLCPCB-Capacitors:0402,10uF
- removed C27, C29, C31, C33, C44, C52: 22uF, PCM_JLCPCB:C_0603, symbol JLCPCB-Capacitors:0603,22uF
- removed C32, C34, C35, C36, C41, C42, C43, C47, C50, C51: 2.2uF, PCM_JLCPCB:C_0402, symbol JLCPCB-Capacitors:0402,2.2uF
- removed C39: 4.7uF, PCM_JLCPCB:C_0402, symbol JLCPCB-Capacitors:0402,4.7uF
- removed D1: 1N4148W, PCM_JLCPCB:D_SOD-123, symbol PCM_JLCPCB-Diodes:Switching,1N4148W
- removed D2, D5, D6, D8: IR, JLCPCB:IR-LED_C131280, symbol JLCPCB-Diodes:LED IR IR26-21c_C131280
- removed D3: White, PCM_JLCPCB:D_0603, symbol JLCPCB-Diodes:LED,0603,White
- removed D4: WS2812B, PCM_JLCPCB:LED-SMD_4P-L1.6-W1.5_XL-1615RGBC-WS2812B, symbol JLCPCB-Extended:LED, WS2812B, 1615
- removed D7: Yellow, PCM_JLCPCB:D_0805, symbol JLCPCB-Diodes:LED,0805,Yellow
- removed D9: Green, PCM_JLCPCB:D_0805, symbol PCM_JLCPCB-Diodes:LED,0805,Green
- removed J1: Connector, USB-TYPE-C-16P, PCM_JLCPCB:TYPE-C-SMD_HX-TYPE-C-16PIN, symbol PCM_JLCPCB-Extended:Connector, USB-TYPE-C-16P
- removed J10, J12, J13, J15, J2, J3, J4, J5, J6, J9: Conn_01x02, Connector_PinHeader_1.00mm:PinHeader_1x02_P1.00mm_Vertical, symbol Connector_Generic:Conn_01x02
- removed J11, J14, J7, J8: Conn_01x03, Connector_PinHeader_2.54mm:PinHeader_1x03_P2.54mm_Vertical, symbol Connector_Generic:Conn_01x03
- removed L3, L4: 2nH, Inductor_SMD:L_0603_1608Metric_Pad1.05x0.95mm_HandSolder, symbol Device:L
- removed L5, L6, L7, L8, L9: 1uH,3.3A, Inductor_SMD:L_1008_2520Metric, symbol JLCPCB-Inductors:1uH,50mA
- removed NTC1: NTC, PCM_JLCPCB:R_0402, symbol JLCPCB-Resistors:0402,10kΩ
- removed Q1, Q2, Q3, Q4, Q5, Q6, Q7: AO3401A, PCM_JLCPCB:Q_SOT-23, symbol PCM_JLCPCB-Transistors:PMOS,AO3401A
- removed R10, R8: 5.1kΩ, PCM_JLCPCB:R_0402, symbol PCM_JLCPCB-Resistors:0402,5.1kΩ
- removed R11, R13: 33Ω, PCM_JLCPCB:R_0402, symbol PCM_JLCPCB-Resistors:0402,33Ω
- removed R12, R15, R38, R6: 100kΩ, PCM_JLCPCB:R_0402, symbol PCM_JLCPCB-Resistors:0402,100kΩ
- removed R14, R16, R18, R20, R24, R26, R30, R34, R39, R7, R9: 10kΩ, PCM_JLCPCB:R_0402, symbol PCM_JLCPCB-Resistors:0402,10kΩ
- removed R17, R19, R23, R25, R31, R33, R35: 10MΩ, PCM_JLCPCB:R_0402, symbol PCM_JLCPCB-Resistors:0402,10MΩ
- removed R21, R22, R27, R29, R32, R36, R37: 1MΩ, PCM_JLCPCB:R_0402, symbol PCM_JLCPCB-Resistors:0402,1MΩ
- removed R28: 22Ω, PCM_JLCPCB:R_0402, symbol PCM_JLCPCB-Resistors:0402,22Ω
- removed TP10, TP11, TP12, TP13, TP14, TP15, TP16, TP17, TP18, TP19, TP20, TP21, TP22, TP23, TP24, TP25, TP26, TP4, TP43, TP44, TP45, TP5, TP6, TP7, TP8, TP9: TestPoint, TestPoint:TestPoint_Pad_D1.0mm, symbol Connector:TestPoint
- removed TP27, TP28, TP29, TP30, TP31, TP32, TP33, TP34, TP35, TP36, TP37, TP38, TP39, TP40, TP41, TP42: TestPoint, Connector_PinHeader_1.00mm:PinHeader_1x01_P1.00mm_Vertical, symbol Connector:TestPoint
- removed TST-R10, TST-R11, TST-R12, TST-R13, TST-R14, TST-R15, TST-R16, TST-R17, TST-R4, TST-R5, TST-R6, TST-R7, TST-R8, TST-R9: 0Ω, PCM_JLCPCB:R_0603, symbol PCM_JLCPCB-Resistors:0603,0Ω
- removed U1: MT9221CT-06BR5, JLCPCB:Current-sensor_MT9221CT-06BR5_C879632, symbol JLCPCB-Extended:Current-sensor_MT9221CT-06BR5_C879632
- removed U3: USBLC6-2SC6, Package_TO_SOT_SMD:SOT-23-6, symbol Power_Protection:USBLC6-2SC6
- removed U4: ESP32-S3, PCM_JLCPCB:QFN-56-1EP_7x7mm_P0.4mm_EP4x4mm_ThermalVias, symbol PCM_JLCPCB-Extended:MCU, ESP32-S3
- removed U5: AXP2101, Package_DFN_QFN:QFN-40-1EP_5x5mm_P0.4mm_EP3.6x3.6mm_ThermalVias, symbol JLCPCB-Extended:AXP2101_C3036461
- removed U6: DS18B20U(UMW), JLCPCB:DS18B20_C695836, symbol JLCPCB-ICs:DS18B20_C695836
- removed U7: W25Q128JVSIQ, PCM_JLCPCB:SOIC-8_L5.3-W5.3-P1.27-LS8.0-BL, symbol PCM_JLCPCB-Memory:16MByte, SPI
- removed Y1: 40MHz, 15pF, JLCPCB:OSC-SMD_4P-L3.2-W2.5-BL_SIT8008BI, symbol JLCPCB-Extended:Crystal, 40MHz, 15pF
- removed Y2: 32.768KHz, Crystal:Crystal_SMD_3215-2Pin_3.2x1.5mm, symbol Device:Crystal
- renumbered C57 to C43, C58 to C44, C59 to C45, C60 to C47, C53 to C66, C56 to C67, C61 to C69, C62 to C70, J18 to J1, J16 to J10, J17 to J2, JP2 to JP1, JP1 to JP3, JP3 to JP4, JP4 to JP5, JP5 to JP6, JP6 to JP7, JP7 to JP8, PB4 to PB1, PB5 to PB2, PB2 to PB4, PB3 to PB5, R43 to R38, R44 to R39, R42 to R43, TP46 to TP1, TP53 to TP47, TP55 to TP49, TP52 to TP56, TP54 to TP57, TP48 to TP63, TP50 to TP64, TP47 to TP66, TP49 to TP67, TP51 to TP85, TST-R20 to TST-R14, TST-R18 to TST-R16, TST-R19 to TST-R18, TST-R21 to TST-R20, TST-R23 to TST-R21, TST-R22 to TST-R26, TST-R24 to TST-R27, U9 to U11, U8 to U15, U10 to U16, U11 to U17
Connections:
- no-connect marks 23 -> 8
Other:
- note removed: "(CL(Load) - Cs(Stray)) * 2 = Capacitance (10p - +/-4p) * 2 = 10p"
- note removed: "2GPIO10"
- note removed: "2GPIO11"
- note removed: "2GPIO12"
- note removed: "2GPIO13"
- note removed: "2GPIO14"
- note removed: "2GPIO15"
- note removed: "2GPIO16"
- note removed: "2GPIO17"
- note removed: "2GPIO18"
- note removed: "2GPIO19"
- note removed: "2GPIO2"
- note removed: "2GPIO20"
- note removed: "2GPIO21"
- note removed: "2GPIO26"
- note removed: "2GPIO27"
- note removed: "2GPIO28"
- note removed: "2GPIO29"
- note removed: "2GPIO30"
- note removed: "2GPIO31"
- note removed: "2GPIO32"
- note removed: "2GPIO33"
- note removed: "2GPIO34"
- note removed: "2GPIO35"
- note removed: "2GPIO36"
- note removed: "2GPIO37"
- note removed: "2GPIO38"
- note removed: "2GPIO4"
- note removed: "2GPIO43"
- note removed: "2GPIO44"
- note removed: "2GPIO5"
- note removed: "2GPIO6"
- note removed: "2GPIO9"
- note removed: "2USB_C"
- note removed: "BATTERY PMU / GUAGE"
- note removed: "Boot Button"
- note removed: "Crystals"
- note removed: "Current Sense"
- note removed: "FC = 1/(2*PI*Rfint*Cfilter) 88Hz = 1/(2*PI*1.8kohm*1nF)"
- note removed: "HSE / LSE"
- note removed: "LIGHTS"
- note removed: "MISC OUTPUTS"
- note removed: "Mode: QuadSPI"
- note removed: "NOR FLASH"
- note removed: "NP = Normal P = Directly in Flash"
- note removed: "NTC wants to be TH11-3H103F while C3018545 is probably a close enough equiv."
- note removed: "OTHER"
- note removed: "PAN"
- note removed: "PCB TEMPERATURE"
- note removed: "PI Filter Antenna"
- note removed: "Pull-Up"
- note removed: "RC SERVO'S"
- note removed: "RF Voltage Filter"
- note removed: "RGB Status LED"
- note removed: "ROTATE"
- note removed: "RST Button"
- note removed: "TILT"
- note removed: "Z=(35+j10)R"
- note removed: "Z=50R"
