File: ESP32S3_Audio_Cam_POE_Medium.kicad_pcb (KiCad board)
At the start: 2 copper layers, 244.5 x 128.3 mm, 241 parts, among them CN1 PJ-316C-6A, J1 Connector, USB-TYPE-C-16P, J10 Conn_01x02, J11 Conn_01x03, J12 Conn_01x02, J13 Conn_01x02, J14 Conn_01x03, J15 Conn_01x02, J16 Conn_01x02, J17 Conn_01x20_Pin, J18 Conn_01x20_Pin, J2 Conn_01x02, J3 Conn_01x02, J4 Conn_01x02, J5 Conn_01x02, J6 Conn_01x02, J7 Conn_01x03, J8 Conn_01x03, J9 Conn_01x02, Q1 AO3401A, Q2 AO3401A, Q3 AO3401A, Q4 AO3401A, Q5 AO3401A, Q6 AO3401A, Q7 AO3401A, U1 MT9221CT-06BR5, U10 ICS-43434, U11 ICS-43434, U3 USBLC6-2SC6, U4 ESP32-S3, U5 AXP2101, U6 DS18B20U(UMW), U7 W25Q128JVSIQ, U8 MAX98357AETE+T, U9 TM1637, Y1 40MHz, 15pF, Y2 32.768KHz

Commit message: Draft Medium
Parts:
- J10, J12, J13, J15, J16, J2, J3, J4, J5, J6, J9: footprint Connector_PinHeader_1.00mm:PinHeader_1x02_P1.00mm_Vertical -> Project-specific:PinHeader_1x02_P1.00mm_Vertical
- TP27, TP28, TP29, TP30, TP31, TP32, TP33, TP34, TP35, TP36, TP37, TP38, TP39, TP40, TP41, TP42, TP46: footprint Connector_PinHeader_1.00mm:PinHeader_1x01_P1.00mm_Vertical -> Project-specific:PinHeader_1x01_P1.00mm_Vertical
- moved C30 168.4 mm to (52.8, 138.8), turned to 0 degrees
- moved C28 165.3 mm to (52.8, 137.5), turned to 0 degrees
- moved TP36 165.3 mm to (57.9, 144.8), turned to 0 degrees
- moved C39 165.1 mm to (54.9, 143.3)
- moved TP28 163.2 mm to (59.9, 144.8), turned to 0 degrees
- moved TP41 162.0 mm to (47.2, 142.9), turned to 0 degrees
- moved C46 161.9 mm to (57.7, 132.6), turned to -90 degrees
- moved C43 161.6 mm to (57.9, 143.3)
- moved C33 160.6 mm to (49.4, 144.4), turned to 180 degrees
- moved L7 160.5 mm to (49.8, 142.2), turned to 0 degrees
- moved TP40 160.3 mm to (56.9, 144.8), turned to 0 degrees
- moved TP39 159.9 mm to (52.8, 144.8), turned to 0 degrees
- moved TP31 159.9 mm to (55.9, 144.8), turned to 0 degrees
- moved C42 159.8 mm to (56.9, 143.3)
- moved TP32 159.4 mm to (61.0, 144.8), turned to 0 degrees
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
Commit message: Draft Medium
Parts:
- moved R36 133.9 mm to (116.8, 118.2)
- moved R24 132.5 mm to (120.6, 120.2), turned to 180 degrees
- moved R34 129.2 mm to (115.6, 120.2), turned to 0 degrees
- moved D5 129.1 mm to (119.4, 122.1), turned to 0 degrees
- moved R33 129.1 mm to (116.2, 115.1), turned to 0 degrees
- moved J2 128.5 mm to (123.8, 120.2), turned to -90 degrees
- moved D2 128.1 mm to (124.5, 122.1), turned to 0 degrees
- moved D8 127.8 mm to (114.3, 122.1), turned to 0 degrees
- moved R17 127.4 mm to (126.4, 115.1), turned to 0 degrees
- moved R18 126.9 mm to (125.7, 120.2), turned to 0 degrees
- moved Q1 124.3 mm to (124.5, 117.6), turned to 180 degrees
- moved J9 124.0 mm to (113.7, 120.2), turned to -90 degrees
- moved R21 123.0 mm to (127.0, 118.2)
- moved TST-R7 121.2 mm to (123.8, 115.1), turned to 180 degrees
- moved R27 119.3 mm to (121.9, 118.2)
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Connections:
- C1 pad 1: VBUS -> VBUS+3V3
- J17 pad 5: +3V3 -> VBUS+3V3
- J4 pad 1: /2U0TXD -> /U0TXD
- J4 pad 2: /2U0RXD -> /U0RXD
- U1 pad 1: Vdrive -> +3V3
- U1 pad 2: Vdrive -> +3V3
- U1 pad 3: VBUS -> VBUS+3V3
- U1 pad 4: VBUS -> VBUS+3V3
- U1 pad 8: VBUS -> VBUS+3V3
- U4 pad 49: /2U0TXD -> /U0TXD
- U4 pad 50: /2U0RXD -> /U0RXD
Routing:
- net +3V3: track 175.2 -> 162.2 mm
- net COM: vias 41 -> 40
Other:
- board size 244.5 x 128.3 mm -> 2.4 x 2.4 mm

Commit message: Draft Medium
Parts:
- moved TST-R12 70.9 mm to (128.3, 153.0)
- moved Q5 70.3 mm to (128.9, 149.9), turned to 0 degrees
- moved R31 69.8 mm to (126.4, 151.1), turned to 90 degrees
- moved R32 66.5 mm to (126.4, 149.2), turned to 90 degrees
- moved C2 65.9 mm to (101.0, 149.9)
- moved U1 65.9 mm to (96.5, 148.6)
- moved J7 60.0 mm to (125.1, 145.9), turned to 90 degrees
- moved C1 59.1 mm to (90.8, 148.6), turned to 90 degrees
- moved J8 53.8 mm to (125.1, 142.1), turned to 90 degrees
- moved TP44 51.7 mm to (120.4, 162.0), turned to 90 degrees
- moved TP24 51.4 mm to (92.7, 140.2), turned to 90 degrees
- moved TP23 50.7 mm to (91.4, 138.3), turned to 90 degrees
- moved R38 50.0 mm to (118.5, 162.0), turned to 180 degrees
- moved R17 48.8 mm to (128.9, 163.8)
- moved R23 48.8 mm to (123.8, 163.8)
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Connections:
- J11 pad 1: /RC.ROT -> /2GPIO40
- J14 pad 1: /RC.OTHR -> /2GPIO39
- J7 pad 1: /RC.PAN -> /2GPIO42
- J8 pad 1: /RC.TILT -> /2GPIO41
- R32 pad 2: /RC.PWR -> /2GPIO45
- TP20 pad 1: /2GPIO39 -> Net-(U4-GPIO9)
- TP21 pad 1: /2GPIO40 -> Net-(U4-GPIO10)
- TP22 pad 1: /2GPIO41 -> Net-(U4-GPIO11)
- TP23 pad 1: /2GPIO42 -> Net-(U4-GPIO12)
- TP24 pad 1: /2GPIO45 -> Net-(U4-GPIO13)
- U4 pad 14: /RC.PWR -> Net-(U4-GPIO9)
- U4 pad 15: /RC.PAN -> Net-(U4-GPIO10)
- U4 pad 16: /RC.TILT -> Net-(U4-GPIO11)
- U4 pad 17: /RC.ROT -> Net-(U4-GPIO12)
- U4 pad 18: /RC.OTHR -> Net-(U4-GPIO13)
Other:
- board size 2.4 x 2.4 mm -> 97.8 x 70.5 mm

Commit message: DRAFT Medium
Parts:
- moved TP17 8.45 mm to (121.3, 152.4)
- moved TST-R17 7.19 mm to (78.7, 144.5), turned to 90 degrees
- moved TP16 6.35 mm to (118.7, 152.4)
- moved TP19 6.27 mm to (123.8, 152.4)
- moved TP15 4.58 mm to (116.2, 152.4)
- moved TP25 4.01 mm to (72.9, 144.7), turned to 0 degrees
- moved U6 3.87 mm to (76.2, 142.6), turned to 180 degrees
- moved TP14 3.81 mm to (113.7, 152.4)
- moved C49 2.57 mm to (78.7, 141.4), turned to -90 degrees
- moved TST-R9 2.26 mm to (70.6, 147.2), turned to 180 degrees
- moved D4 2.26 mm to (70.6, 144.0), turned to 0 degrees
- moved C35 1.97 mm to (47.0, 144.8)
- moved C36 1.97 mm to (48.0, 144.8)
- moved C42 1.97 mm to (51.1, 144.8)
- moved C43 1.97 mm to (52.1, 144.8)
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Routing:
- net /PMU.Vsys: track 0.00 -> 65.0 mm, vias 0 -> 10
- net +3V3: track 162.2 -> 209.9 mm
- net COM: track 36.1 -> 74.3 mm, vias 40 -> 59
- net Net-(J12-Pin_1): track 0.00 -> 24.0 mm
- net /RF2: track 0.00 -> 23.4 mm
- net /RC.VDD: track 0.00 -> 16.3 mm
- net VBUS+3V3: track 0.00 -> 15.9 mm
- net Net-(PB1-A): track 0.00 -> 14.0 mm
- net /PMU.Vo4: track 0.00 -> 12.0 mm
- net /PMU.Vo2: track 0.00 -> 11.1 mm
- net /VDCDC5: track 0.00 -> 10.7 mm
- net /PMU.Vo3: track 0.00 -> 9.12 mm
- net Net-(J13-Pin_1): track 0.00 -> 8.45 mm
- net Net-(U5-CHGLED): track 0.00 -> 8.36 mm
- net Net-(U5-FB1): track 0.00 -> 7.79 mm
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